Commit message: Add Gazebo plugins and launch files for Barracuda robot simulation

File: urdf/barracuda.xacro (robot description, xacro)
@@ -33,4 +33,46 @@
     </joint>
     <gazebo>
+        <plugin name="uuv_plugin" filename="libuuv_underwater_object_ros_plugin.so">
+            <!-- Hydro parameters for the vehicle-->
+            <fluid_density>1028.0</fluid_density>
+            <flow_velocity_topic>hydrodynamics/current_velocity</flow_velocity_topic>
+            <debug>$(arg debug)</debug>
+            <link name="$(arg namespace)/base_link">
+            <neutrally_buoyant>1</neutrally_buoyant>
+            <!-- See eNovus technical specifications -->
+            <volume>1.8382</volume> <!-- This is a guess (similar size to Smilodon but heavier) -->
+            <box>
+                <width>1.6</width>
+                <length>2.7</length>
+                <height>1.8</height>
+            </box>
+            <!-- Center of buoyancy is a guess, using same value as RexRov -->
+            <center_of_buoyancy>0.0 0.0 0.3</center_of_buoyancy>
+            <hydrodynamic_model>
+                <type>fossen</type>
+                <!-- Everything else in the model is pulled straight from Berg2012
+                    (which means it's not even close for this vehicle) -->
+                <!-- Added mass: see p.28 in Berg2012 -->
+                <added_mass>
+                779.79 -6.8773 -103.32  8.5426 -165.54 -7.8033
+                -6.8773    1222   51.29  409.44 -5.8488  62.726
+                -103.32   51.29  3659.9  6.1112 -386.42  10.774
+                8.5426  409.44  6.1112   534.9 -10.027  21.019
+                -165.54 -5.8488 -386.42 -10.027  842.69 -1.1162
+                -7.8033  62.726  10.775  21.019 -1.1162  224.32
+                </added_mass>
+                <!-- Linear damping: see p.31 in Berg2012 -->
+                <linear_damping>
+                -74.82 -69.48 -728.4 -268.8 -309.77 -105
+                </linear_damping>
+                <!-- Non-linear damping: see p.30 in Berg2012 -->
+                <quadratic_damping>
+                -748.22 -992.53 -1821.01 -672 -774.44 -523.27
+                </quadratic_damping>
+            </hydrodynamic_model>
+            </link>
+        </plugin>
+    </gazebo>
+    <gazebo>
         <plugin name="gazebo_ros_control" filename="libgazebo_ros_control.so">
             <robotNamespace>$(arg namespace)</robotNamespace>

Commit message: Update Barracuda launch and URDF files for namespace consistency and IMU sensor integration

File: urdf/barracuda.xacro (robot description, xacro)
@@ -1,8 +1,7 @@
 <?xml version="1.0"?>
 <robot name="barracuda" xmlns:xacro="http://www.ros.org/wiki/xacro">
-   <!-- "Dummy" base link to eliminate root link inertia warning -->
-    <xacro:include filename="$(find barracuda_description)/urdf/sensors.xacro"/>
     <xacro:arg name="debug" default="0"/>
     <xacro:arg name="namespace" default="barracuda"/>
+    <!-- "Dummy" base link to eliminate root link inertia warning -->
     <link name="$(arg namespace)/base_link"/>
     <link name="$(arg namespace)/barracuda_link">
@@ -33,5 +32,6 @@
         <child link="$(arg namespace)/barracuda_link"/>
     </joint>
-    <xacro:imu_sensor parent_link="barracuda_link" imu_name="imu" namespace="$(arg namespace)"/>
+    <xacro:include filename="$(find barracuda_description)/urdf/sensors.xacro"/>
+    <xacro:imu_sensor parent_link="$(arg namespace)/barracuda_link" imu_name="imu" namespace="$(arg namespace)"/>
     <gazebo>
         <plugin name="uuv_plugin" filename="libuuv_underwater_object_ros_plugin.so">
@@ -79,5 +79,5 @@
         <plugin name="gazebo_ros_control" filename="libgazebo_ros_control.so">
             <robotNamespace>$(arg namespace)</robotNamespace>
-            <robotParam>$(arg namespace)</robotParam>
+            <robotParam>/robot_description</robotParam>
         </plugin>
     </gazebo>

File: urdf/sensors.xacro (robot description, xacro)
@@ -2,16 +2,16 @@
 <robot xmlns:xacro="http://www.ros.org/wiki/xacro">
   <!-- Macro for the IMU -->
-  <xacro:macro name="imu_sensor" params="parent_link imu_name">
+  <xacro:macro name="imu_sensor" params="parent_link imu_name namespace">
     <!-- IMU Link -->
-    <link name="${imu_name}_link">
+    <link name="${namespace}/${imu_name}_link">
     </link>
     <!-- Fixed Joint to Attach the IMU -->
-    <joint name="${imu_name}_joint" type="fixed">
-      <parent>${parent_link}</parent>
-      <child>${imu_name}_link</child>
+    <joint name="${namespace}/${imu_name}_joint" type="fixed">
+      <parent link="${parent_link}"/>
+      <child link="${namespace}/${imu_name}_link"/>
       <origin xyz="0 0 0.1" rpy="0 0 0"/>
     </joint>
     <!-- IMU Sensor -->
-    <gazebo reference="${imu_name}_link">
+    <gazebo reference="${namespace}/${imu_name}_link">
       <gravity>true</gravity>
       <sensor name="${imu_name}_sensor" type="imu">
@@ -19,13 +19,13 @@
         <update_rate>100</update_rate>
         <visualize>true</visualize>
-        <topic>imu/data</topic>
+        <topic>${namespace}/${imu_name}/data</topic>
         <plugin filename="libgazebo_ros_imu_sensor.so" name="${imu_name}_plugin">
-          <topicName>$(arg namespace)/${imu_name}/data</topicName>
-          <bodyName>${imu_name}_link</bodyName>
+          <topicName>${namespace}/${imu_name}/data</topicName>
+          <bodyName>${namespace}/${imu_name}_link</bodyName>
           <updateRateHZ>100.0</updateRateHZ>
-          <gaussianNoise>0.0</gaussianNoise>
+          <gaussianNoise>2e-4</gaussianNoise>
           <xyzOffset>0 0 0</xyzOffset>
           <rpyOffset>0 0 0</rpyOffset>
-          <frameName>${imu_name}_link</frameName>
+          <frameName>${namespace}/${imu_name}_link</frameName>
           <initialOrientationAsReference>false</initialOrientationAsReference>
         </plugin>

Commit message: add thruster template code

File: urdf/barracuda.xacro (robot description, xacro)
@@ -3,4 +3,7 @@
     <xacro:arg name="debug" default="0"/>
     <xacro:arg name="namespace" default="barracuda"/>
+    <xacro:include filename="$(find uuv_descriptions)/urdf/common.urdf.xacro"/>
+    <xacro:include filename="$(find uuv_gazebo_ros_plugins)/urdf/thruster_snippets.xacro"/>
+    <xacro:property name="prop_mesh_file" value="file://$(find barracuda_description)/meshes/t100_thruster.dae"/>
     <!-- "Dummy" base link to eliminate root link inertia warning -->
     <link name="$(arg namespace)/base_link"/>
@@ -79,7 +82,42 @@
         <plugin name="gazebo_ros_control" filename="libgazebo_ros_control.so">
             <robotNamespace>$(arg namespace)</robotNamespace>
-            <robotParam>/robot_description</robotParam>
+            <robotParam>$(arg namespace)/robot_description</robotParam>
         </plugin>
     </gazebo>
+    <!-- FROM MANTARAY NEED CHANGE -->
+    <xacro:macro name="thruster_macro" params="thruster_id *origin">
+        <xacro:thruster_module_first_order_basic_fcn_macro
+            namespace="$(arg namespace)"
+            thruster_id="${thruster_id}"
+            mesh_filename="${prop_mesh_file}"
+            dyn_time_constant="0.05"
+            rotor_constant="0.00031">
+            <xacro:insert_block name="origin"/>
+        </xacro:thruster_module_first_order_basic_fcn_macro>
+    </xacro:macro>
+    <xacro:thruster_macro thruster_id="0">
+      <origin xyz="-0.25 -0.333 0.145" rpy="${90*d2r} 0 ${300*d2r}"/>
+    </xacro:thruster_macro>
+    <xacro:thruster_macro thruster_id="1">
+      <origin xyz="0.25 -0.333 0.145" rpy="${90*d2r} 0 ${240*d2r}"/>
+    </xacro:thruster_macro>
+    <xacro:thruster_macro thruster_id="2">
+      <origin xyz="0.25 0.333 0.145" rpy="${90*d2r} 0 ${120*d2r}"/>
+    </xacro:thruster_macro>
+    <xacro:thruster_macro thruster_id="3">
+      <origin xyz="-0.25 0.3333 0.145" rpy="${90*d2r} 0 ${60*d2r}"/>
+    </xacro:thruster_macro>
+    <xacro:thruster_macro thruster_id="4">
+      <origin xyz="-0.25 0.19 0.19" rpy="0 ${90*d2r} 0"/>
+    </xacro:thruster_macro>
+    <xacro:thruster_macro thruster_id="5">
+      <origin xyz="0.25 0.19 0.19" rpy="0 ${90*d2r} 0"/>
+    </xacro:thruster_macro>
+    <xacro:thruster_macro thruster_id="6">
+      <origin xyz="-0.25 -0.19 0.19" rpy="0 ${90*d2r} 0"/>
+    </xacro:thruster_macro>
+    <xacro:thruster_macro thruster_id="7">
+      <origin xyz="0.25 -0.19 0.19" rpy="0 ${90*d2r} 0"/>
+    </xacro:thruster_macro>
     <!-- Default joint state publisher -->
     <gazebo>

Commit message: added new thruster

File: urdf/barracuda.xacro (robot description, xacro)
@@ -5,5 +5,5 @@
     <xacro:include filename="$(find uuv_descriptions)/urdf/common.urdf.xacro"/>
     <xacro:include filename="$(find uuv_gazebo_ros_plugins)/urdf/thruster_snippets.xacro"/>
-    <xacro:property name="prop_mesh_file" value="file://$(find barracuda_description)/meshes/t100_thruster.dae"/>
+    <xacro:property name="prop_mesh_file" value="file://$(find barracuda_description)/meshes/T200-THRUSTER-R1.STL"/>
     <!-- "Dummy" base link to eliminate root link inertia warning -->
     <link name="$(arg namespace)/base_link"/>

Commit message: t100

File: urdf/barracuda.xacro (robot description, xacro)
@@ -5,5 +5,5 @@
     <xacro:include filename="$(find uuv_descriptions)/urdf/common.urdf.xacro"/>
     <xacro:include filename="$(find uuv_gazebo_ros_plugins)/urdf/thruster_snippets.xacro"/>
-    <xacro:property name="prop_mesh_file" value="file://$(find barracuda_description)/meshes/T200-THRUSTER-R1.STL"/>
+    <xacro:property name="prop_mesh_file" value="file://$(find barracuda_description)/meshes/t200_thruster.dae"/>
     <!-- "Dummy" base link to eliminate root link inertia warning -->
     <link name="$(arg namespace)/base_link"/>

Commit message: Add initial depth camera and DVL macros

File: urdf/barracuda.xacro (robot description, xacro)
@@ -37,4 +37,6 @@
     <xacro:include filename="$(find barracuda_description)/urdf/sensors.xacro"/>
     <xacro:imu_sensor parent_link="$(arg namespace)/barracuda_link" imu_name="imu" namespace="$(arg namespace)"/>
+    <xacro:dvl parent_link="$(arg namespace)/barracuda_link" dvl_name="dvl" namespace="$(arg namespace)"/>
+    <!-- <xacro:depth_camera parent_link="$(arg namespace)/barracuda_link" namespace="$(arg namespace)"/> -->
     <gazebo>
         <plugin name="uuv_plugin" filename="libuuv_underwater_object_ros_plugin.so">

File: urdf/sensors.xacro (robot description, xacro)
@@ -8,7 +8,7 @@
     <!-- Fixed Joint to Attach the IMU -->
     <joint name="${namespace}/${imu_name}_joint" type="fixed">
-      <parent link="${parent_link}"/>
-      <child link="${namespace}/${imu_name}_link"/>
-      <origin xyz="0 0 0.1" rpy="0 0 0"/>
+      <parent link="${parent_link}" />
+      <child link="${namespace}/${imu_name}_link" />
+      <origin xyz="0 0 0.1" rpy="0 0 0" />
     </joint>
     <!-- IMU Sensor -->
@@ -33,3 +33,104 @@
     </gazebo>
   </xacro:macro>
+  <!-- Macro for single sonar for the DVL  -->
+  <xacro:macro name="dvl_single_sonar" params="namespace dvl_name index pitch yaw update_rate">
+    <link name="${namespace}/${dvl_name}_sonar${index}_link">
+    </link>
+    <joint name="${namespace}/${dvl_name}_sonar${index}_joint" type="revolute">
+      <origin xyz="0 0 0" rpy="0 ${pitch} ${yaw}"/>
+      <parent link="${namespace}/${dvl_name}_link"/>
+      <child link="${namespace}/${dvl_name}_sonar${index}_link"/>
+      <limit upper="0" lower="0" effort="0" velocity="0"/>
+      <axis xyz="1 0 0"/>
+    </joint>
+    <gazebo reference="${namespace}/${dvl_name}_sonar${index}_link">
+      <sensor type="ray" name="${dvl_name}_sonar${index}">
+        <pose>0 0 0 0 0 0</pose>
+        <update_rate>${update_rate}</update_rate>
+        <visualize>true</visualize>
+        <ray>
+          <scan>
+            <horizontal>
+              <samples>3</samples>
+              <resolution>1</resolution>
+              <min_angle>-0.025</min_angle>
+              <max_angle>0.025</max_angle>
+            </horizontal>
+            <vertical>
+              <samples>3</samples>
+              <resolution>1</resolution>
+              <min_angle>-0.025</min_angle>
+              <max_angle>0.025</max_angle>
+            </vertical>
+          </scan>
+          <range>
+            <min>0.2</min>
+            <max>75</max>
+            <resolution>0.01</resolution>
+          </range>
+        </ray>
+        <plugin name="${dvl_name}_sonar${index}" filename="libgazebo_ros_range.so">
+          <gaussianNoise>0.005</gaussianNoise>
+          <alwaysOn>true</alwaysOn>
+          <updateRate>${update_rate}</updateRate>
+          <topicName>${namespace}/${dvl_name}_sonar${index}</topicName>
+          <frameName>${namespace}/${dvl_name}_sonar${index}_link</frameName>
+          <fov>0.05</fov>
+          <radiation>ultrasound</radiation>
+        </plugin>
+      </sensor>
+    </gazebo>
+  </xacro:macro>
+  <!-- Macro for the DVL -->
+  <xacro:macro name="dvl" params="parent_link dvl_name namespace">
+    <!-- DVL Link -->
+    <link name="${namespace}/${dvl_name}_link">
+    </link>
+    <!-- Fixed joint to attach the DVL-->
+    <joint name="${namespace}/${dvl_name}_joint" type="fixed">
+      <parent link="${parent_link}" />
+      <child link="${namespace}/${dvl_name}_link" />
+      <origin xyz="0 0 0" rpy="0 0 0" />
+    </joint>
+    <!-- DVL sonars -->
+    <xacro:dvl_single_sonar
+      namespace="${namespace}" dvl_name="${dvl_name}"
+      index="0" pitch="-0.4363" yaw="0.0" update_rate="7">
+    </xacro:dvl_single_sonar>
+    <xacro:dvl_single_sonar
+      namespace="${namespace}" dvl_name="${dvl_name}"
+      index="1" pitch="0.0" yaw="0.4363" update_rate="7">
+    </xacro:dvl_single_sonar>
+    <xacro:dvl_single_sonar
+      namespace="${namespace}" dvl_name="${dvl_name}"
+      index="2" pitch="0.4363" yaw="0.0" update_rate="7">
+    </xacro:dvl_single_sonar>
+    <xacro:dvl_single_sonar
+      namespace="${namespace}" dvl_name="${dvl_name}"
+      index="3" pitch="0.0" yaw="-0.4363" update_rate="7">
+    </xacro:dvl_single_sonar>
+    <!-- DVL Sensor-->
+    <gazebo reference="${namespace}/${dvl_name}_link">
+      <plugin name="libuuv_gazebo_dvl_plugin" filename="libuuv_gazebo_ros_dvl_plugin.so">
+        <robot_namespace>${namespace}</robot_namespace>	<!-- ROS topic & link namespace -->
+        <sensor_topic>${dvl_name}</sensor_topic> 		<!-- name of the sensor data ROS topic -->
+        <update_rate>7</update_rate>		<!-- Hertz (should match beam plugin specs) -->
+        <noise_sigma>0.005</noise_sigma>		<!-- Only used for coviariance matrix -->
+        <noise_amplitude>0.005</noise_amplitude>	<!-- Gaussian noise added to velocity vector components -->
+        <enable_gazebo_messages>false</enable_gazebo_messages>
+        <enable_local_ned_frame>false</enable_local_ned_frame>  <!-- Can use if a global NED frame is available -->
+        <static_reference_frame>world</static_reference_frame>
+        <!-- Declaring the links associated with individual sonar beams (see below)-->
+        <beam_link_name_0>${namespace}/${dvl_name}_sonar0_link</beam_link_name_0>
+        <beam_link_name_1>${namespace}/${dvl_name}_sonar1_link</beam_link_name_1>
+        <beam_link_name_2>${namespace}/${dvl_name}_sonar2_link</beam_link_name_2>
+        <beam_link_name_3>${namespace}/${dvl_name}_sonar3_link</beam_link_name_3>
+        <!-- Declaring the individual sonar beam output ROS range topics -->
+        <beam_topic_0>${dvl_name}_sonar0</beam_topic_0>
+        <beam_topic_1>${dvl_name}_sonar1</beam_topic_1>
+        <beam_topic_2>${dvl_name}_sonar2</beam_topic_2>
+        <beam_topic_3>${dvl_name}_sonar3</beam_topic_3>
+      </plugin>
+    </gazebo>
+  </xacro:macro>
 </robot>

Commit message: Update mesh references in barracuda.xacro to use the correct DAE file

File: urdf/barracuda.xacro (robot description, xacro)
@@ -20,5 +20,5 @@
             <origin xyz="0 0 0" rpy="0 0 1.5708"/>
             <geometry>
-                <mesh filename="file://$(find barracuda_description)/meshes/mantaray_base_link.stl" scale="1 1 1"/>
+                <mesh filename="file://$(find barracuda_description)/meshes/barracuda_base_link.dae" scale="1 1 1"/>
             </geometry>
         </visual>
@@ -26,5 +26,5 @@
             <origin xyz="0 0 0" rpy="0 0 1.5708"/>
             <geometry>
-                <mesh filename="file://$(find barracuda_description)/meshes/mantaray_base_link.stl" scale="1 1 1"/>
+                <mesh filename="file://$(find barracuda_description)/meshes/barracuda_base_link.dae" scale="1 1 1"/>
             </geometry>
         </collision>

Commit message: thrusters added correctly

File: urdf/barracuda.xacro (robot description, xacro)
@@ -96,27 +96,35 @@
         </xacro:thruster_module_first_order_basic_fcn_macro>
     </xacro:macro>
+    <!--right top-->
+    <xacro:thruster_macro thruster_id="8">
+      <origin xyz="0.0 -0.322 0.0767" rpy="${90*d2r} ${90*d2r} 0"/>
+    </xacro:thruster_macro>
+    <!--right mid-->
+    <xacro:thruster_macro thruster_id="9">
+      <origin xyz="0.00525 -0.43515 0.0" rpy="${90*d2r} 0 0"/>
+    </xacro:thruster_macro>
+    <!--left top-->
     <xacro:thruster_macro thruster_id="0">
-      <origin xyz="-0.25 -0.333 0.145" rpy="${90*d2r} 0 ${300*d2r}"/>
+      <origin xyz="0.0 0.322 0.0767" rpy="${-90*d2r} ${90*d2r} 0"/>
     </xacro:thruster_macro>
+    <!--left mid-->
     <xacro:thruster_macro thruster_id="1">
-      <origin xyz="0.25 -0.333 0.145" rpy="${90*d2r} 0 ${240*d2r}"/>
+      <origin xyz="0.00525 0.43515 0.0" rpy="${90*d2r} 0 ${180*d2r}"/>
     </xacro:thruster_macro>
+    <!--front left-->
     <xacro:thruster_macro thruster_id="2">
-      <origin xyz="0.25 0.333 0.145" rpy="${90*d2r} 0 ${120*d2r}"/>
+      <origin xyz="0.30916 0.36341 0.0" rpy="${-90*d2r} ${135*d2r} ${-48.49*d2r}"/>
     </xacro:thruster_macro>
+    <!--back left-->
     <xacro:thruster_macro thruster_id="3">
-      <origin xyz="-0.25 0.3333 0.145" rpy="${90*d2r} 0 ${60*d2r}"/>
+      <origin xyz="-0.30916 0.36341 0.0" rpy="${-90*d2r} ${45*d2r} ${48.49*d2r}"/>
     </xacro:thruster_macro>
+    <!--front right-->
     <xacro:thruster_macro thruster_id="4">
-      <origin xyz="-0.25 0.19 0.19" rpy="0 ${90*d2r} 0"/>
+      <origin xyz="0.30916 -0.36341 0.0" rpy="${90*d2r} ${135*d2r} ${48.49*d2r}"/>
     </xacro:thruster_macro>
+    <!--back right-->
     <xacro:thruster_macro thruster_id="5">
-      <origin xyz="0.25 0.19 0.19" rpy="0 ${90*d2r} 0"/>
-    </xacro:thruster_macro>
-    <xacro:thruster_macro thruster_id="6">
-      <origin xyz="-0.25 -0.19 0.19" rpy="0 ${90*d2r} 0"/>
-    </xacro:thruster_macro>
-    <xacro:thruster_macro thruster_id="7">
-      <origin xyz="0.25 -0.19 0.19" rpy="0 ${90*d2r} 0"/>
+      <origin xyz="-0.30916 -0.36341 0.0" rpy="${-45*d2r} ${45*d2r} ${-48.49*d2r}"/>
     </xacro:thruster_macro>
     <!-- Default joint state publisher -->
