Commit message: DVL URDF working

File: urdf/barracuda.xacro (robot description, xacro)
@@ -37,6 +37,7 @@
     <xacro:include filename="$(find barracuda_description)/urdf/sensors.xacro"/>
     <xacro:imu_sensor parent_link="$(arg namespace)/barracuda_link" imu_name="imu" namespace="$(arg namespace)"/>
-    <xacro:dvl parent_link="$(arg namespace)/barracuda_link" dvl_name="dvl" namespace="$(arg namespace)"/>
-    <!-- <xacro:depth_camera parent_link="$(arg namespace)/barracuda_link" namespace="$(arg namespace)"/> -->
+    <xacro:dvl parent_link="$(arg namespace)/base_link" dvl_name="dvl" namespace="$(arg namespace)"/>
+    <xacro:include filename="$(find barracuda_description)/urdf/depth_camera.xacro"/>
+    <xacro:depth_camera parent_link="$(arg namespace)/barracuda_link" namespace="$(arg namespace)"/>
     <gazebo>
         <plugin name="uuv_plugin" filename="libuuv_underwater_object_ros_plugin.so">

File: urdf/sensors.xacro (robot description, xacro)
@@ -36,11 +36,17 @@
   <xacro:macro name="dvl_single_sonar" params="namespace dvl_name index pitch yaw update_rate">
     <link name="${namespace}/${dvl_name}_sonar${index}_link">
+      <inertial>
+        <mass value="0.001" />
+        <origin xyz="0 0 0" rpy="0 0 0" />
+        <inertia ixx="0.000000017" ixy="0" ixz="0" iyy="0.000000017" iyz="0" izz="0.000000017" />
+      </inertial>
+      <!-- <xacro:no_collision /> -->
     </link>
     <joint name="${namespace}/${dvl_name}_sonar${index}_joint" type="revolute">
-      <origin xyz="0 0 0" rpy="0 ${pitch} ${yaw}"/>
-      <parent link="${namespace}/${dvl_name}_link"/>
-      <child link="${namespace}/${dvl_name}_sonar${index}_link"/>
-      <limit upper="0" lower="0" effort="0" velocity="0"/>
-      <axis xyz="1 0 0"/>
+      <origin xyz="0 0 0" rpy="0 ${pitch} ${yaw}" />
+      <parent link="${namespace}/${dvl_name}_link" />
+      <child link="${namespace}/${dvl_name}_sonar${index}_link" />
+      <limit upper="0" lower="0" effort="0" velocity="0" />
+      <axis xyz="1 0 0" />
     </joint>
     <gazebo reference="${namespace}/${dvl_name}_sonar${index}_link">
@@ -70,5 +76,5 @@
           </range>
         </ray>
-        <plugin name="${dvl_name}_sonar${index}" filename="libgazebo_ros_range.so">
+        <plugin filename="libgazebo_ros_range.so" name="${dvl_name}_sonar${index}">
           <gaussianNoise>0.005</gaussianNoise>
           <alwaysOn>true</alwaysOn>
@@ -86,4 +92,22 @@
     <!-- DVL Link -->
     <link name="${namespace}/${dvl_name}_link">
+      <inertial>
+        <mass value="8.8" />
+        <origin xyz="0 0 0" rpy="0 0 0" />
+        <inertia ixx="0.071732122" ixy="0" ixz="0" iyy="0.071732122" iyz="0" izz="0.055786544" />
+      </inertial>
+      <visual>
+        <geometry>
+          <mesh
+            filename="package://dave_sensor_models/models/teledyne_whn_uuvsim/meshes/WorkhorseNavigator.dae" />
+        </geometry>
+        <origin xyz="0 0 0" rpy="0 1.5707963267948966 0" />
+      </visual>
+      <collision>
+        <geometry>
+          <cylinder length="0.2445" radius="0.1126" />
+        </geometry>
+        <origin xyz="0 0 0" rpy="0 1.5707963267948966 0" />
+      </collision>
     </link>
     <!-- Fixed joint to attach the DVL-->
@@ -112,12 +136,16 @@
     <!-- DVL Sensor-->
     <gazebo reference="${namespace}/${dvl_name}_link">
-      <plugin name="libuuv_gazebo_dvl_plugin" filename="libuuv_gazebo_ros_dvl_plugin.so">
+      <plugin filename="libuuv_gazebo_ros_dvl_plugin.so" name="libuuv_gazebo_dvl_plugin">
         <robot_namespace>${namespace}</robot_namespace>	<!-- ROS topic & link namespace -->
+        <link_name>${parent_link}</link_name> <!-- (string, required): name of the body which holds
+        the IMU sensor -->
         <sensor_topic>${dvl_name}</sensor_topic> 		<!-- name of the sensor data ROS topic -->
         <update_rate>7</update_rate>		<!-- Hertz (should match beam plugin specs) -->
         <noise_sigma>0.005</noise_sigma>		<!-- Only used for coviariance matrix -->
-        <noise_amplitude>0.005</noise_amplitude>	<!-- Gaussian noise added to velocity vector components -->
+        <noise_amplitude>0.005</noise_amplitude>	<!-- Gaussian noise added to velocity vector
+        components -->
         <enable_gazebo_messages>false</enable_gazebo_messages>
-        <enable_local_ned_frame>false</enable_local_ned_frame>  <!-- Can use if a global NED frame is available -->
+        <enable_local_ned_frame>false</enable_local_ned_frame>  <!-- Can use if a global NED frame is
+        available -->
         <static_reference_frame>world</static_reference_frame>
         <!-- Declaring the links associated with individual sonar beams (see below)-->

Commit message: Update mesh file references in barracuda.xacro to use STL format

File: urdf/barracuda.xacro (robot description, xacro)
@@ -20,5 +20,5 @@
             <origin xyz="0 0 0" rpy="0 0 1.5708"/>
             <geometry>
-                <mesh filename="file://$(find barracuda_description)/meshes/barracuda_base_link.dae" scale="1 1 1"/>
+                <mesh filename="file://$(find barracuda_description)/meshes/barracuda_base_link.stl" scale="1 1 1"/>
             </geometry>
         </visual>
@@ -26,5 +26,5 @@
             <origin xyz="0 0 0" rpy="0 0 1.5708"/>
             <geometry>
-                <mesh filename="file://$(find barracuda_description)/meshes/barracuda_base_link.dae" scale="1 1 1"/>
+                <mesh filename="file://$(find barracuda_description)/meshes/barracuda_base_link.stl" scale="1 1 1"/>
             </geometry>
         </collision>

Commit message: Update barracuda.xacro

File: urdf/barracuda.xacro (robot description, xacro)
@@ -18,5 +18,5 @@
         </inertial>
         <visual>
-            <origin xyz="0 0 0" rpy="0 0 1.5708"/>
+            <origin xyz="0 0 0" rpy="0 0 0"/>
             <geometry>
                 <mesh filename="file://$(find barracuda_description)/meshes/barracuda_base_link.stl" scale="1 1 1"/>
@@ -24,5 +24,5 @@
         </visual>
         <collision>
-            <origin xyz="0 0 0" rpy="0 0 1.5708"/>
+            <origin xyz="0 0 0" rpy="0 0 0"/>
             <geometry>
                 <mesh filename="file://$(find barracuda_description)/meshes/barracuda_base_link.stl" scale="1 1 1"/>

Commit message: Update barracuda.xacro

File: urdf/barracuda.xacro (robot description, xacro)
@@ -20,5 +20,5 @@
             <origin xyz="0 0 0" rpy="0 0 0"/>
             <geometry>
-                <mesh filename="file://$(find barracuda_description)/meshes/barracuda_base_link.stl" scale="1 1 1"/>
+                <mesh filename="file://$(find barracuda_description)/meshes/barracuda_base_link.dae" scale="1 1 1"/>
             </geometry>
         </visual>
@@ -26,5 +26,5 @@
             <origin xyz="0 0 0" rpy="0 0 0"/>
             <geometry>
-                <mesh filename="file://$(find barracuda_description)/meshes/barracuda_base_link.stl" scale="1 1 1"/>
+                <mesh filename="file://$(find barracuda_description)/meshes/barracuda_base_link.dae" scale="1 1 1"/>
             </geometry>
         </collision>

Commit message: fixed center and thruster position

File: urdf/barracuda.xacro (robot description, xacro)
@@ -97,33 +97,33 @@
     </xacro:macro>
     <!--right top-->
-    <xacro:thruster_macro thruster_id="8">
-      <origin xyz="0.0 -0.322 0.0767" rpy="${90*d2r} ${90*d2r} 0"/>
+    <xacro:thruster_macro thruster_id="0">
+      <origin xyz="0.0 -0.322 0.1535" rpy="${90*d2r} ${90*d2r} 0"/>
     </xacro:thruster_macro>
     <!--right mid-->
-    <xacro:thruster_macro thruster_id="9">
+    <xacro:thruster_macro thruster_id="1">
       <origin xyz="0.00525 -0.43515 0.0" rpy="${90*d2r} 0 0"/>
     </xacro:thruster_macro>
     <!--left top-->
-    <xacro:thruster_macro thruster_id="0">
-      <origin xyz="0.0 0.322 0.0767" rpy="${-90*d2r} ${90*d2r} 0"/>
+    <xacro:thruster_macro thruster_id="2">
+      <origin xyz="0.0 0.322 0.1535" rpy="${-90*d2r} ${90*d2r} 0"/>
     </xacro:thruster_macro>
     <!--left mid-->
-    <xacro:thruster_macro thruster_id="1">
+    <xacro:thruster_macro thruster_id="3">
       <origin xyz="0.00525 0.43515 0.0" rpy="${90*d2r} 0 ${180*d2r}"/>
     </xacro:thruster_macro>
     <!--front left-->
-    <xacro:thruster_macro thruster_id="2">
+    <xacro:thruster_macro thruster_id="4">
       <origin xyz="0.30916 0.36341 0.0" rpy="${-90*d2r} ${135*d2r} ${-48.49*d2r}"/>
     </xacro:thruster_macro>
     <!--back left-->
-    <xacro:thruster_macro thruster_id="3">
+    <xacro:thruster_macro thruster_id="5">
       <origin xyz="-0.30916 0.36341 0.0" rpy="${-90*d2r} ${45*d2r} ${48.49*d2r}"/>
     </xacro:thruster_macro>
     <!--front right-->
-    <xacro:thruster_macro thruster_id="4">
+    <xacro:thruster_macro thruster_id="6">
       <origin xyz="0.30916 -0.36341 0.0" rpy="${90*d2r} ${135*d2r} ${48.49*d2r}"/>
     </xacro:thruster_macro>
     <!--back right-->
-    <xacro:thruster_macro thruster_id="5">
+    <xacro:thruster_macro thruster_id="7">
       <origin xyz="-0.30916 -0.36341 0.0" rpy="${-45*d2r} ${45*d2r} ${-48.49*d2r}"/>
     </xacro:thruster_macro>

Commit message: base mesh orientation fix

File: urdf/barracuda.xacro (robot description, xacro)
@@ -18,5 +18,5 @@
         </inertial>
         <visual>
-            <origin xyz="0 0 0" rpy="0 0 0"/>
+            <origin xyz="0 0 0" rpy="0 0 ${90*d2r}"/>
             <geometry>
                 <mesh filename="file://$(find barracuda_description)/meshes/barracuda_base_link.dae" scale="1 1 1"/>
@@ -24,5 +24,5 @@
         </visual>
         <collision>
-            <origin xyz="0 0 0" rpy="0 0 0"/>
+            <origin xyz="0 0 0" rpy="0 0 ${90*d2r}"/>
             <geometry>
                 <mesh filename="file://$(find barracuda_description)/meshes/barracuda_base_link.dae" scale="1 1 1"/>

Commit message: Finalize sensors

File: urdf/barracuda.xacro (robot description, xacro)
@@ -37,5 +37,5 @@
     <xacro:include filename="$(find barracuda_description)/urdf/sensors.xacro"/>
     <xacro:imu_sensor parent_link="$(arg namespace)/barracuda_link" imu_name="imu" namespace="$(arg namespace)"/>
-    <xacro:dvl parent_link="$(arg namespace)/base_link" dvl_name="dvl" namespace="$(arg namespace)"/>
+    <xacro:dvl parent_link="$(arg namespace)/base_link" dvl_name="dvl" namespace="$(arg namespace)" />
     <xacro:include filename="$(find barracuda_description)/urdf/depth_camera.xacro"/>
     <xacro:depth_camera parent_link="$(arg namespace)/barracuda_link" namespace="$(arg namespace)"/>

File: urdf/depth_camera.xacro (robot description, xacro)
@@ -34,7 +34,7 @@
     <link name="${namespace}/$(arg camera_name)_camera_center">
       <visual>
-        <origin xyz="${screw_offset_x} 0 ${screw_offset_z}" rpy="0 0 0" />
+        <origin xyz="${screw_offset_x} 0 ${screw_offset_z}" rpy="0 0 -${M_PI/2}" />
         <geometry>
-          <mesh filename="file://$(find barracuda_description)/meshes/$(arg camera_model).stl" />
+          <mesh filename="file://$(find barracuda_description)/meshes/$(arg camera_model).dae" />
         </geometry>
         <material name="zedm_mat">
@@ -76,57 +76,4 @@
     <!-- Stereo Camera -->
     <gazebo reference="${namespace}/$(arg camera_name)_left_camera_frame">
-      <!-- <sensor type="multicamera" name="stereo_camera">
-        <update_rate>10.0</update_rate>
-        <camera name="left">
-          <horizontal_fov>1.089</horizontal_fov>
-          <image>
-            <width>1920</width>
-            <height>1080</height>
-            <format>R8G8B8</format>
-          </image>
-          <clip>
-            <near>0.04</near>
-            <far>100</far>
-          </clip>
-          <noise>
-            <type>gaussian</type>
-            <mean>0.0</mean>
-            <stddev>0.007</stddev>
-          </noise>
-        </camera>
-        <camera name="right">
-          <pose>0 0 0 0 0 0</pose>
-          <horizontal_fov>1.089</horizontal_fov>
-          <image>
-            <width>1920</width>
-            <height>1080</height>
-            <format>R8G8B8</format>
-          </image>
-          <clip>
-            <near>0.04</near>
-            <far>100</far>
-          </clip>
-          <noise>
-            <type>gaussian</type>
-            <mean>0.0</mean>
-            <stddev>0.007</stddev>
-          </noise>
-        </camera>
-        <plugin name="stereo_camera_controller" filename="libgazebo_ros_multicamera.so">
-          <alwaysOn>true</alwaysOn>
-          <updateRate>0.0</updateRate>
-          <cameraName>multisense_sl/camera</cameraName>
-          <imageTopicName>image_raw</imageTopicName>
-          <cameraInfoTopicName>camera_info</cameraInfoTopicName>
-          <frameName>${namespace}/$(arg camera_name)_left_camera_optical_frame</frameName>
-          <rightFrameName>${namespace}/$(arg camera_name)_right_camera_optical_frame</rightFrameName>
-          <hackBaseline>0.07</hackBaseline>
-          <distortionK1>0.0</distortionK1>
-          <distortionK2>0.0</distortionK2>
-          <distortionK3>0.0</distortionK3>
-          <distortionT1>0.0</distortionT1>
-          <distortionT2>0.0</distortionT2>
-        </plugin>
-      </sensor> -->
       <sensor name="left_camera" type="depth">
         <pose>0 0 0 0 0 0</pose>
@@ -146,16 +93,15 @@
           </clip>
         </camera>
-        <plugin name="depth_camera_controller" filename="libgazebo_ros_depth_camera.so"
-          frame_name="${namespace}/$(arg camera_name)_left_camera_optical_frame">
+        <plugin name="depth_camera_controller" filename="libgazebo_ros_depth_camera.so">
           <alwaysOn>true</alwaysOn>
           <min_depth>0.1</min_depth>
           <max_depth>100.0</max_depth>
-          <attenuationR>0.01</attenuationR>
+          <!-- <attenuationR>0.01</attenuationR>
           <attenuationG>0.01</attenuationG>
-          <attenuationB>0.003</attenuationB>
-          <backgroundR>0</backgroundR>
+          <attenuationB>0.003</attenuationB> -->
+          <!-- <backgroundR>0</backgroundR>
           <backgroundG>0</backgroundG>
-          <backgroundB>0</backgroundB>
-          <!-- <robotNamespace>${namespace}</robotNamespace> -->
+          <backgroundB>0</backgroundB> -->
+          <robotNamespace>${namespace}</robotNamespace>
           <updateRate>10.0</updateRate>
           <frameName>${namespace}/$(arg camera_name)_left_camera_optical_frame</frameName>
@@ -167,5 +113,32 @@
       </sensor>
     </gazebo>
-    <!-- Depth Camera -->
+    <gazebo reference="$(arg namespace)/$(arg camera_name)_right_camera_frame">
+      <sensor name="right_camera" type="camera">
+        <pose>0 0 0 0 0 0</pose>
+        <visualize>true</visualize>
+        <update_rate>10</update_rate>
+        <camera>
+          <camera_name>${namespace}/$(arg camera_name)_right_camera_frame</camera_name>
+          <horizontal_fov>1.089</horizontal_fov> <!-- Need to change -->
+          <image>
+            <format>R8G8B8</format> <!-- Need to change -->
+            <width>1920</width>
+            <height>1080</height>
+          </image>
+          <clip> <!-- Minimum and maximum range the camera can see -->
+            <near>0.04</near>
+            <far>100.0</far>
+          </clip>
+        </camera>
+        <plugin name="camera_controller" filename="libgazebo_ros_camera.so">
+          <alwaysOn>true</alwaysOn>
+          <updateRate>10.0</updateRate>
+          <robotNamespace>${namespace}</robotNamespace>
+          <frameName>${namespace}/$(arg camera_name)_right_camera_optical_frame</frameName>
+          <cameraName>${namespace}/right_camera</cameraName>
+          <imageTopicName>right_camera_image</imageTopicName>
+        </plugin>
+      </sensor>
+    </gazebo>
   </xacro:macro>
 </robot>

File: urdf/sensors.xacro (robot description, xacro)
@@ -10,5 +10,5 @@
       <parent link="${parent_link}" />
       <child link="${namespace}/${imu_name}_link" />
-      <origin xyz="0 0 0.1" rpy="0 0 0" />
+      <origin xyz="0 0 0" rpy="0 0 0" />
     </joint>
     <!-- IMU Sensor -->
@@ -41,5 +41,4 @@
         <inertia ixx="0.000000017" ixy="0" ixz="0" iyy="0.000000017" iyz="0" izz="0.000000017" />
       </inertial>
-      <!-- <xacro:no_collision /> -->
     </link>
     <joint name="${namespace}/${dvl_name}_sonar${index}_joint" type="revolute">
@@ -71,6 +70,6 @@
           </scan>
           <range>
-            <min>0.2</min>
-            <max>75</max>
+            <min>0.05</min>
+            <max>50</max>
             <resolution>0.01</resolution>
           </range>
@@ -93,5 +92,5 @@
     <link name="${namespace}/${dvl_name}_link">
       <inertial>
-        <mass value="8.8" />
+        <mass value="0.105" />
         <origin xyz="0 0 0" rpy="0 0 0" />
         <inertia ixx="0.071732122" ixy="0" ixz="0" iyy="0.071732122" iyz="0" izz="0.055786544" />
@@ -99,6 +98,7 @@
       <visual>
         <geometry>
-          <mesh
-            filename="package://dave_sensor_models/models/teledyne_whn_uuvsim/meshes/WorkhorseNavigator.dae" />
+          <mesh filename="file://$(find barracuda_description)/meshes/dvl.dae" >
+            <pose>0 0 0  0 1.5707963267948966 0</pose>
+          </mesh>
         </geometry>
         <origin xyz="0 0 0" rpy="0 1.5707963267948966 0" />
@@ -106,5 +106,5 @@
       <collision>
         <geometry>
-          <cylinder length="0.2445" radius="0.1126" />
+          <cylinder length="0.025" radius="0.033" />
         </geometry>
         <origin xyz="0 0 0" rpy="0 1.5707963267948966 0" />
@@ -115,25 +115,25 @@
       <parent link="${parent_link}" />
       <child link="${namespace}/${dvl_name}_link" />
-      <origin xyz="0 0 0" rpy="0 0 0" />
+      <origin xyz="0 0 -0.5" rpy="0 ${0.5*pi} 0" />
     </joint>
     <!-- DVL sonars -->
     <xacro:dvl_single_sonar
       namespace="${namespace}" dvl_name="${dvl_name}"
-      index="0" pitch="-0.4363" yaw="0.0" update_rate="7">
+      index="0" pitch="-0.4363" yaw="0.0" update_rate="10">
     </xacro:dvl_single_sonar>
     <xacro:dvl_single_sonar
       namespace="${namespace}" dvl_name="${dvl_name}"
-      index="1" pitch="0.0" yaw="0.4363" update_rate="7">
+      index="1" pitch="0.0" yaw="0.4363" update_rate="10">
     </xacro:dvl_single_sonar>
     <xacro:dvl_single_sonar
       namespace="${namespace}" dvl_name="${dvl_name}"
-      index="2" pitch="0.4363" yaw="0.0" update_rate="7">
+      index="2" pitch="0.4363" yaw="0.0" update_rate="10">
     </xacro:dvl_single_sonar>
     <xacro:dvl_single_sonar
       namespace="${namespace}" dvl_name="${dvl_name}"
-      index="3" pitch="0.0" yaw="-0.4363" update_rate="7">
+      index="3" pitch="0.0" yaw="-0.4363" update_rate="10">
     </xacro:dvl_single_sonar>
     <!-- DVL Sensor-->
-    <gazebo reference="${namespace}/${dvl_name}_link">
+    <gazebo>
       <plugin filename="libuuv_gazebo_ros_dvl_plugin.so" name="libuuv_gazebo_dvl_plugin">
         <robot_namespace>${namespace}</robot_namespace>	<!-- ROS topic & link namespace -->
@@ -141,5 +141,5 @@
         the IMU sensor -->
         <sensor_topic>${dvl_name}</sensor_topic> 		<!-- name of the sensor data ROS topic -->
-        <update_rate>7</update_rate>		<!-- Hertz (should match beam plugin specs) -->
+        <update_rate>10</update_rate>		<!-- Hertz (should match beam plugin specs) -->
         <noise_sigma>0.005</noise_sigma>		<!-- Only used for coviariance matrix -->
         <noise_amplitude>0.005</noise_amplitude>	<!-- Gaussian noise added to velocity vector

Commit message: Adjust sensor positions

File: urdf/barracuda.xacro (robot description, xacro)
@@ -85,5 +85,5 @@
         <plugin name="gazebo_ros_control" filename="libgazebo_ros_control.so">
             <robotNamespace>$(arg namespace)</robotNamespace>
-            <robotParam>$(arg namespace)/robot_description</robotParam>
+            <robotParam>robot_description</robotParam>
         </plugin>
     </gazebo>

File: urdf/depth_camera.xacro (robot description, xacro)
@@ -6,10 +6,10 @@
     <xacro:arg name="camera_name" default="zed" />
     <xacro:arg name="camera_model" default="zedm" />
-    <xacro:arg name="cam_pos_x" default="0.0" />
-    <xacro:arg name="cam_pos_y" default="0.4" />
-    <xacro:arg name="cam_pos_z" default="0.2" />
+    <xacro:arg name="cam_pos_x" default="-0.3" />
+    <xacro:arg name="cam_pos_y" default="0.0" />
+    <xacro:arg name="cam_pos_z" default="0.0" />
     <xacro:arg name="cam_roll" default="0.0" />
     <xacro:arg name="cam_pitch" default="0.0" />
-    <xacro:arg name="cam_yaw" default="${M_PI/2}" />
+    <xacro:arg name="cam_yaw" default="${M_PI}" />
     <!-- <xacro:arg name="frame_id" value="${namespace}/base_link" /> -->
     <xacro:arg name="gnss_frame" default="" />

File: urdf/sensors.xacro (robot description, xacro)
@@ -115,5 +115,5 @@
       <parent link="${parent_link}" />
       <child link="${namespace}/${dvl_name}_link" />
-      <origin xyz="0 0 -0.5" rpy="0 ${0.5*pi} 0" />
+      <origin xyz="0 0 -0.15" rpy="0 ${0.5*pi} 0" />
     </joint>
     <!-- DVL sonars -->
