Commit message: allow specification of parent link

File: urdf/barracuda.xacro (robot description, xacro)
@@ -95,4 +95,5 @@
             namespace="$(arg namespace)"
             thruster_id="${thruster_id}"
+            parent_link="$(arg namespace)/barracuda_link"
             mesh_filename="${prop_mesh_file}"
             dyn_time_constant="0.05"
@@ -107,5 +108,5 @@
     <!--right mid-->
     <xacro:thruster_macro thruster_id="1">
-      <origin xyz="0.00525 -0.43515 0.0" rpy="${90*d2r} 0 0"/>
+      <origin xyz="0.00525 -0.43515 0.0" rpy="${90*d2r} 0 ${180*d2r}"/>
     </xacro:thruster_macro>
     <!--left top-->
@@ -115,5 +116,5 @@
     <!--left mid-->
     <xacro:thruster_macro thruster_id="3">
-      <origin xyz="0.00525 0.43515 0.0" rpy="${90*d2r} 0 0"/>
+      <origin xyz="0.00525 0.43515 0.0" rpy="${90*d2r} 0 ${180*d2r}"/>
     </xacro:thruster_macro>
     <!--front left-->

File: urdf/thruster_snippets.xacro (robot description, xacro)
@@ -72,4 +72,5 @@
     params="namespace
             thruster_id
+            parent_link
             *origin
             mesh_filename
@@ -79,5 +80,5 @@
       <xacro:insert_block name="origin"/>
       <axis xyz="1 0 0"/>
-      <parent link="${namespace}/base_link"/>
+      <parent link="${parent_link}"/>
       <child link="${namespace}/thruster_${thruster_id}"/>
     </joint>
@@ -122,4 +123,5 @@
       params="namespace
               thruster_id
+              parent_link
               *origin
               mesh_filename
@@ -129,4 +131,5 @@
       namespace="${namespace}"
       thruster_id="${thruster_id}"
+      parent_link="${parent_link}"
       mesh_filename="${mesh_filename}">
       <xacro:insert_block name="origin"/>

Commit message: Update barracuda.xacro

File: urdf/barracuda.xacro (robot description, xacro)
@@ -10,5 +10,5 @@
     <link name="$(arg namespace)/barracuda_link">
         <inertial>
-            <origin xyz="0 0 0" rpy="0 0 ${180*d2r}"/>
+            <origin xyz="0 0 0" rpy="0 0 0"/>
             <mass value="36.3"/>
             <inertia

Commit message: Update barracuda.xacro

File: urdf/barracuda.xacro (robot description, xacro)
@@ -18,5 +18,5 @@
         </inertial>
         <visual>
-            <origin xyz="0 0 0" rpy="0 0 ${90*d2r}"/>
+            <origin xyz="0 0 0" rpy="0 0 ${-90*d2r}"/>
             <geometry>
                 <mesh filename="file://$(find barracuda_description)/meshes/barracuda_base_link.dae" scale="1 1 1"/>
@@ -24,5 +24,5 @@
         </visual>
         <collision>
-            <origin xyz="0 0 0" rpy="0 0 ${90*d2r}"/>
+            <origin xyz="0 0 0" rpy="0 0 ${-90*d2r}"/>
             <geometry>
                 <mesh filename="file://$(find barracuda_description)/meshes/barracuda_base_link.dae" scale="1 1 1"/>
@@ -104,33 +104,33 @@
     <!--right top-->
     <xacro:thruster_macro thruster_id="0">
-      <origin xyz="0.0 -0.322 0.1535" rpy="${90*d2r} ${90*d2r} 0"/>
+      <origin xyz="0.0 0.322 0.1535" rpy="${90*d2r} ${90*d2r} ${180*d2r}"/>
     </xacro:thruster_macro>
     <!--right mid-->
     <xacro:thruster_macro thruster_id="1">
-      <origin xyz="0.00525 -0.43515 0.0" rpy="${90*d2r} 0 ${180*d2r}"/>
+      <origin xyz="-0.00525 0.43515 0.0" rpy="${90*d2r} 0 0"/>
     </xacro:thruster_macro>
     <!--left top-->
     <xacro:thruster_macro thruster_id="2">
-      <origin xyz="0.0 0.322 0.1535" rpy="${-90*d2r} ${90*d2r} 0"/>
+      <origin xyz="0.0 -0.322 0.1535" rpy="${-90*d2r} ${90*d2r} ${180*d2r}"/>
     </xacro:thruster_macro>
     <!--left mid-->
     <xacro:thruster_macro thruster_id="3">
-      <origin xyz="0.00525 0.43515 0.0" rpy="${90*d2r} 0 ${180*d2r}"/>
+      <origin xyz="-0.00525 -0.43515 0.0" rpy="${90*d2r} 0 0"/>
     </xacro:thruster_macro>
     <!--front left-->
     <xacro:thruster_macro thruster_id="4">
-      <origin xyz="0.30916 0.36341 0.0" rpy="${-90*d2r} ${135*d2r} ${-48.49*d2r}"/>
+      <origin xyz="-0.30916 -0.36341 0.0" rpy="${-90*d2r} ${135*d2r} ${131.51*d2r}"/>
     </xacro:thruster_macro>
     <!--back left-->
     <xacro:thruster_macro thruster_id="5">
-      <origin xyz="-0.30916 0.36341 0.0" rpy="${-90*d2r} ${45*d2r} ${48.49*d2r}"/>
+      <origin xyz="0.30916 -0.36341 0.0" rpy="${-90*d2r} ${45*d2r} ${-131.51*d2r}"/>
     </xacro:thruster_macro>
     <!--front right-->
     <xacro:thruster_macro thruster_id="6">
-      <origin xyz="0.30916 -0.36341 0.0" rpy="${90*d2r} ${135*d2r} ${48.49*d2r}"/>
+      <origin xyz="-0.30916 0.36341 0.0" rpy="${90*d2r} ${135*d2r} ${-131.51*d2r}"/>
     </xacro:thruster_macro>
     <!--back right-->
     <xacro:thruster_macro thruster_id="7">
-      <origin xyz="-0.30916 -0.36341 0.0" rpy="${-45*d2r} ${45*d2r} ${-48.49*d2r}"/>
+      <origin xyz="0.30916 0.36341 0.0" rpy="${-45*d2r} ${45*d2r} ${131.51*d2r}"/>
     </xacro:thruster_macro>
     <!-- Default joint state publisher -->

Commit message: Update barracuda.xacro

File: urdf/barracuda.xacro (robot description, xacro)
@@ -108,5 +108,5 @@
     <!--right mid-->
     <xacro:thruster_macro thruster_id="1">
-      <origin xyz="-0.00525 0.43515 0.0" rpy="${90*d2r} 0 0"/>
+      <origin xyz="-0.00525 0.43515 0.0" rpy="${90*d2r} 0 ${180*d2r}"/>
     </xacro:thruster_macro>
     <!--left top-->
@@ -116,5 +116,5 @@
     <!--left mid-->
     <xacro:thruster_macro thruster_id="3">
-      <origin xyz="-0.00525 -0.43515 0.0" rpy="${90*d2r} 0 0"/>
+      <origin xyz="-0.00525 -0.43515 0.0" rpy="${90*d2r} 0 ${180*d2r}"/>
     </xacro:thruster_macro>
     <!--front left-->

Commit message: Make thrusters tf tree parent barracuda_link, make front of robot point forward (#22)
* Update barracuda.xacro

* Update depth_camera.xacro

* Update barracuda.xacro

File: urdf/barracuda.xacro (robot description, xacro)
@@ -18,5 +18,5 @@
         </inertial>
         <visual>
-            <origin xyz="0 0 0" rpy="0 0 ${90*d2r}"/>
+            <origin xyz="0 0 0" rpy="0 0 ${-90*d2r}"/>
             <geometry>
                 <mesh filename="file://$(find barracuda_description)/meshes/barracuda_base_link.dae" scale="1 1 1"/>
@@ -24,5 +24,5 @@
         </visual>
         <collision>
-            <origin xyz="0 0 0" rpy="0 0 ${90*d2r}"/>
+            <origin xyz="0 0 0" rpy="0 0 ${-90*d2r}"/>
             <geometry>
                 <mesh filename="file://$(find barracuda_description)/meshes/barracuda_base_link.dae" scale="1 1 1"/>
@@ -104,33 +104,33 @@
     <!--right top-->
     <xacro:thruster_macro thruster_id="0">
-      <origin xyz="0.0 -0.322 0.1535" rpy="${90*d2r} ${90*d2r} 0"/>
+      <origin xyz="0.0 0.322 0.1535" rpy="${90*d2r} ${90*d2r} ${180*d2r}"/>
     </xacro:thruster_macro>
     <!--right mid-->
     <xacro:thruster_macro thruster_id="1">
-      <origin xyz="0.00525 -0.43515 0.0" rpy="${90*d2r} 0 ${180*d2r}"/>
+      <origin xyz="-0.00525 0.43515 0.0" rpy="${90*d2r} 0 ${180*d2r}"/>
     </xacro:thruster_macro>
     <!--left top-->
     <xacro:thruster_macro thruster_id="2">
-      <origin xyz="0.0 0.322 0.1535" rpy="${-90*d2r} ${90*d2r} 0"/>
+      <origin xyz="0.0 -0.322 0.1535" rpy="${-90*d2r} ${90*d2r} ${180*d2r}"/>
     </xacro:thruster_macro>
     <!--left mid-->
     <xacro:thruster_macro thruster_id="3">
-      <origin xyz="0.00525 0.43515 0.0" rpy="${90*d2r} 0 ${180*d2r}"/>
+      <origin xyz="-0.00525 -0.43515 0.0" rpy="${90*d2r} 0 ${180*d2r}"/>
     </xacro:thruster_macro>
     <!--front left-->
     <xacro:thruster_macro thruster_id="4">
-      <origin xyz="0.30916 0.36341 0.0" rpy="${-90*d2r} ${135*d2r} ${-48.49*d2r}"/>
+      <origin xyz="-0.30916 -0.36341 0.0" rpy="${-90*d2r} ${135*d2r} ${131.51*d2r}"/>
     </xacro:thruster_macro>
     <!--back left-->
     <xacro:thruster_macro thruster_id="5">
-      <origin xyz="-0.30916 0.36341 0.0" rpy="${-90*d2r} ${45*d2r} ${48.49*d2r}"/>
+      <origin xyz="0.30916 -0.36341 0.0" rpy="${-90*d2r} ${45*d2r} ${-131.51*d2r}"/>
     </xacro:thruster_macro>
     <!--front right-->
     <xacro:thruster_macro thruster_id="6">
-      <origin xyz="0.30916 -0.36341 0.0" rpy="${90*d2r} ${135*d2r} ${48.49*d2r}"/>
+      <origin xyz="-0.30916 0.36341 0.0" rpy="${90*d2r} ${135*d2r} ${-131.51*d2r}"/>
     </xacro:thruster_macro>
     <!--back right-->
     <xacro:thruster_macro thruster_id="7">
-      <origin xyz="-0.30916 -0.36341 0.0" rpy="${-45*d2r} ${45*d2r} ${-48.49*d2r}"/>
+      <origin xyz="0.30916 0.36341 0.0" rpy="${-45*d2r} ${45*d2r} ${131.51*d2r}"/>
     </xacro:thruster_macro>
     <!-- Default joint state publisher -->
