Commit message: Revert "update to remove slash from tf prefix"
This reverts commit b279062f0dcac603ad9eb52451bc7b70cea25d2b.

File: urdf/barracuda.xacro (robot description, xacro)
@@ -7,6 +7,6 @@
     <xacro:property name="prop_mesh_file" value="file://$(find barracuda_description)/meshes/t200_thruster.dae"/>
     <!-- "Dummy" base link to eliminate root link inertia warning -->
-    <link name="base_link"/>
-    <link name="$(arg namespace)_barracuda_link">
+    <link name="$(arg namespace)/base_link"/>
+    <link name="$(arg namespace)/barracuda_link">
         <inertial>
             <origin xyz="0 0 0" rpy="0 0 0"/>
@@ -30,16 +30,16 @@
         </collision>
     </link>
-    <joint name="$(arg namespace)_barracuda_base_joint" type="fixed">
+    <joint name="$(arg namespace)/barracuda_base_joint" type="fixed">
         <origin xyz="0 0 0" rpy="0 0 0"/>
-        <parent link="base_link"/>
-        <child link="$(arg namespace)_barracuda_link"/>
+        <parent link="$(arg namespace)/base_link"/>
+        <child link="$(arg namespace)/barracuda_link"/>
     </joint>
     <xacro:include filename="$(find barracuda_description)/urdf/sensors.xacro"/>
-    <xacro:imu_sensor parent_link="$(arg namespace)_barracuda_link" imu_name="imu" namespace="$(arg namespace)"/>
-    <xacro:dvl parent_link="base_link" dvl_name="dvl" namespace="$(arg namespace)" />
-    <xacro:lidar parent_link="$(arg namespace)_barracuda_link" lidar_name="ping360" namespace="$(arg namespace)" />
-    <xacro:altimeter parent_link="$(arg namespace)_barracuda_link" altimeter_name="ping1d" namespace="$(arg namespace)" />
+    <xacro:imu_sensor parent_link="$(arg namespace)/barracuda_link" imu_name="imu" namespace="$(arg namespace)"/>
+    <xacro:dvl parent_link="$(arg namespace)/base_link" dvl_name="dvl" namespace="$(arg namespace)" />
+    <xacro:lidar parent_link="$(arg namespace)/barracuda_link" lidar_name="ping360" namespace="$(arg namespace)" />
+    <xacro:altimeter parent_link="$(arg namespace)/barracuda_link" altimeter_name="ping1d" namespace="$(arg namespace)" />
     <xacro:include filename="$(find barracuda_description)/urdf/depth_camera.xacro"/>
-    <xacro:depth_camera parent_link="$(arg namespace)_barracuda_link" namespace="$(arg namespace)"/>
+    <xacro:depth_camera parent_link="$(arg namespace)/barracuda_link" namespace="$(arg namespace)"/>
     <gazebo>
         <plugin name="uuv_plugin" filename="libuuv_underwater_object_ros_plugin.so">
@@ -48,5 +48,5 @@
             <flow_velocity_topic>hydrodynamics/current_velocity</flow_velocity_topic>
             <debug>$(arg debug)</debug>
-            <link name="base_link">
+            <link name="$(arg namespace)/base_link">
             <neutrally_buoyant>1</neutrally_buoyant>
             <!-- See eNovus technical specifications -->
@@ -95,5 +95,5 @@
             namespace="$(arg namespace)"
             thruster_id="${thruster_id}"
-            parent_link="$(arg namespace)_barracuda_link"
+            parent_link="$(arg namespace)/barracuda_link"
             mesh_filename="${prop_mesh_file}"
             dyn_time_constant="0.05"

File: urdf/depth_camera.xacro (robot description, xacro)
@@ -12,9 +12,9 @@
     <xacro:arg name="cam_pitch" default="0.0" />
     <xacro:arg name="cam_yaw" default="0.0" />
-    <!-- <xacro:arg name="frame_id" value="base_link" /> -->
+    <!-- <xacro:arg name="frame_id" value="${namespace}/base_link" /> -->
     <xacro:arg name="gnss_frame" default="" />
     <!-- <xacro:property name="parent_link" default="" /> -->
-    <!-- <xacro:property name="parent" value="base_link" /> -->
-    <xacro:property name="frame_id" value="base_link" />
+    <!-- <xacro:property name="parent" value="${namespace}/base_link" /> -->
+    <xacro:property name="frame_id" value="${namespace}/base_link" />
     <xacro:property name="baseline" value="0.06" />
     <xacro:property name="height" value="0.0265" />
@@ -25,12 +25,12 @@
     <joint name="$(arg camera_name)_base_joint" type="fixed">
       <parent link="${parent_link}" />
-      <child link="${namespace}_$(arg camera_name)_base_link" />
+      <child link="${namespace}/$(arg camera_name)_base_link" />
       <origin xyz="$(arg cam_pos_x) $(arg cam_pos_y) $(arg cam_pos_z)"
         rpy="$(arg cam_roll) $(arg cam_pitch) $(arg cam_yaw)" />
     </joint>
     <!-- Camera Link -->
-    <link name="${namespace}_$(arg camera_name)_base_link" />
+    <link name="${namespace}/$(arg camera_name)_base_link" />
     <!-- Camera Center -->
-    <link name="${namespace}_$(arg camera_name)_camera_center">
+    <link name="${namespace}/$(arg camera_name)_camera_center">
       <visual>
         <origin xyz="${screw_offset_x} 0 ${screw_offset_z}" rpy="0 0 -${M_PI/2}" />
@@ -44,36 +44,36 @@
     </link>
     <joint name="$(arg camera_name)_camera_center_joint" type="fixed">
-      <parent link="${namespace}_$(arg camera_name)_base_link" />
-      <child link="${namespace}_$(arg camera_name)_camera_center" />
+      <parent link="${namespace}/$(arg camera_name)_base_link" />
+      <child link="${namespace}/$(arg camera_name)_camera_center" />
       <origin xyz="0 0 ${height/2}" rpy="0 ${bottom_slope} 0" />
     </joint>
     <!-- Left Camera -->
-    <link name="${namespace}_$(arg camera_name)_left_camera_frame" />
+    <link name="${namespace}/$(arg camera_name)_left_camera_frame" />
     <joint name="$(arg camera_name)_left_camera_joint" type="fixed">
-      <parent link="${namespace}_$(arg camera_name)_camera_center" />
-      <child link="${namespace}_$(arg camera_name)_left_camera_frame" />
+      <parent link="${namespace}/$(arg camera_name)_camera_center" />
+      <child link="${namespace}/$(arg camera_name)_left_camera_frame" />
       <origin xyz="${optical_offset_x} ${baseline/2} 0" rpy="0 0 0" />
     </joint>
-    <link name="${namespace}_$(arg camera_name)_left_camera_optical_frame" />
+    <link name="${namespace}/$(arg camera_name)_left_camera_optical_frame" />
     <joint name="$(arg camera_name)_left_camera_optical_joint" type="fixed">
       <origin xyz="0 0 0" rpy="-${M_PI/2} 0.0 -${M_PI/2}" />
-      <parent link="${namespace}_$(arg camera_name)_left_camera_frame" />
-      <child link="${namespace}_$(arg camera_name)_left_camera_optical_frame" />
+      <parent link="${namespace}/$(arg camera_name)_left_camera_frame" />
+      <child link="${namespace}/$(arg camera_name)_left_camera_optical_frame" />
     </joint>
     <!-- Right Camera -->
-    <link name="${namespace}_$(arg camera_name)_right_camera_frame" />
+    <link name="${namespace}/$(arg camera_name)_right_camera_frame" />
     <joint name="$(arg camera_name)_right_camera_joint" type="fixed">
-      <parent link="${namespace}_$(arg camera_name)_camera_center" />
-      <child link="${namespace}_$(arg camera_name)_right_camera_frame" />
+      <parent link="${namespace}/$(arg camera_name)_camera_center" />
+      <child link="${namespace}/$(arg camera_name)_right_camera_frame" />
       <origin xyz="${optical_offset_x} -${baseline/2} 0" rpy="0 0 0" />
     </joint>
-    <link name="${namespace}_$(arg camera_name)_right_camera_optical_frame" />
+    <link name="${namespace}/$(arg camera_name)_right_camera_optical_frame" />
     <joint name="$(arg camera_name)_right_camera_optical_joint" type="fixed">
       <origin xyz="0 0 0" rpy="-${M_PI/2} 0.0 -${M_PI/2}" />
-      <parent link="${namespace}_$(arg camera_name)_right_camera_frame" />
-      <child link="${namespace}_$(arg camera_name)_right_camera_optical_frame" />
+      <parent link="${namespace}/$(arg camera_name)_right_camera_frame" />
+      <child link="${namespace}/$(arg camera_name)_right_camera_optical_frame" />
     </joint>
     <!-- Stereo Camera -->
-    <gazebo reference="${namespace}_$(arg camera_name)_left_camera_frame">
+    <gazebo reference="${namespace}/$(arg camera_name)_left_camera_frame">
       <sensor name="left_camera" type="depth">
         <pose>0 0 0 0 0 0</pose>
@@ -81,5 +81,5 @@
         <update_rate>15</update_rate>
         <camera>
-          <camera_name>${namespace}_$(arg camera_name)_left_camera_frame</camera_name>
+          <camera_name>${namespace}/$(arg camera_name)_left_camera_frame</camera_name>
           <horizontal_fov>1.089</horizontal_fov> <!-- Need to change -->
           <image>
@@ -105,5 +105,5 @@
           <robotNamespace>${namespace}</robotNamespace>
           <updateRate>15.0</updateRate>
-          <frameName>${namespace}_$(arg camera_name)_left_camera_optical_frame</frameName>
+          <frameName>${namespace}/$(arg camera_name)_left_camera_optical_frame</frameName>
           <cameraName>left_camera</cameraName>
           <imageTopicName>left_camera_image</imageTopicName>
@@ -113,5 +113,5 @@
       </sensor>
     </gazebo>
-    <gazebo reference="$(arg namespace)_$(arg camera_name)_right_camera_frame">
+    <gazebo reference="$(arg namespace)/$(arg camera_name)_right_camera_frame">
       <sensor name="right_camera" type="camera">
         <pose>0 0 0 0 0 0</pose>
@@ -119,5 +119,5 @@
         <update_rate>15</update_rate>
         <camera>
-          <camera_name>${namespace}_$(arg camera_name)_right_camera_frame</camera_name>
+          <camera_name>${namespace}/$(arg camera_name)_right_camera_frame</camera_name>
           <horizontal_fov>1.089</horizontal_fov> <!-- Need to change -->
           <image>
@@ -135,5 +135,5 @@
           <updateRate>15.0</updateRate>
           <robotNamespace>${namespace}</robotNamespace>
-          <frameName>${namespace}_$(arg camera_name)_right_camera_optical_frame</frameName>
+          <frameName>${namespace}/$(arg camera_name)_right_camera_optical_frame</frameName>
           <cameraName>right_camera</cameraName>
           <imageTopicName>right_camera_image</imageTopicName>

File: urdf/sensors.xacro (robot description, xacro)
@@ -4,14 +4,14 @@
   <xacro:macro name="imu_sensor" params="parent_link imu_name namespace">
     <!-- IMU Link -->
-    <link name="${namespace}_${imu_name}_link">
+    <link name="${namespace}/${imu_name}_link">
     </link>
     <!-- Fixed Joint to Attach the IMU -->
-    <joint name="${namespace}_${imu_name}_joint" type="fixed">
-      <parent link="${parent_link}" />
-      <child link="${namespace}_${imu_name}_link" />
+    <joint name="${namespace}/${imu_name}_joint" type="fixed">
+      <parent link="${parent_link}" />
+      <child link="${namespace}/${imu_name}_link" />
       <origin xyz="0 0 0" rpy="0 0 0" />
     </joint>
     <!-- IMU Sensor -->
-    <gazebo reference="${namespace}_${imu_name}_link">
+    <gazebo reference="${namespace}/${imu_name}_link">
       <gravity>true</gravity>
       <sensor name="${imu_name}_sensor" type="imu">
@@ -22,10 +22,10 @@
         <plugin filename="libgazebo_ros_imu_sensor.so" name="${imu_name}_plugin">
           <topicName>${namespace}/${imu_name}/data</topicName>
-          <bodyName>${namespace}_${imu_name}_link</bodyName>
+          <bodyName>${namespace}/${imu_name}_link</bodyName>
           <updateRateHZ>100.0</updateRateHZ>
           <gaussianNoise>2e-4</gaussianNoise>
           <xyzOffset>0 0 0</xyzOffset>
           <rpyOffset>0 0 0</rpyOffset>
-          <frameName>${namespace}_${imu_name}_link</frameName>
+          <frameName>${namespace}/${imu_name}_link</frameName>
           <initialOrientationAsReference>false</initialOrientationAsReference>
         </plugin>
@@ -35,5 +35,5 @@
   <!-- Macro for single sonar for the DVL  -->
   <xacro:macro name="dvl_single_sonar" params="namespace dvl_name index pitch yaw update_rate">
-    <link name="${namespace}_${dvl_name}_sonar${index}_link">
+    <link name="${namespace}/${dvl_name}_sonar${index}_link">
       <inertial>
         <mass value="0.001" />
@@ -42,12 +42,12 @@
       </inertial>
     </link>
-    <joint name="${namespace}_${dvl_name}_sonar${index}_joint" type="revolute">
+    <joint name="${namespace}/${dvl_name}_sonar${index}_joint" type="revolute">
       <origin xyz="0 0 0" rpy="0 ${pitch} ${yaw}" />
-      <parent link="${namespace}_${dvl_name}_link" />
-      <child link="${namespace}_${dvl_name}_sonar${index}_link" />
+      <parent link="${namespace}/${dvl_name}_link" />
+      <child link="${namespace}/${dvl_name}_sonar${index}_link" />
       <limit upper="0" lower="0" effort="0" velocity="0" />
       <axis xyz="1 0 0" />
     </joint>
-    <gazebo reference="${namespace}_${dvl_name}_sonar${index}_link">
+    <gazebo reference="${namespace}/${dvl_name}_sonar${index}_link">
       <sensor type="ray" name="${dvl_name}_sonar${index}">
         <pose>0 0 0 0 0 0</pose>
@@ -80,5 +80,5 @@
           <updateRate>${update_rate}</updateRate>
           <topicName>${namespace}/${dvl_name}_sonar${index}</topicName>
-          <frameName>${namespace}_${dvl_name}_sonar${index}_link</frameName>
+          <frameName>${namespace}/${dvl_name}_sonar${index}_link</frameName>
           <fov>0.05</fov>
           <radiation>ultrasound</radiation>
@@ -90,5 +90,5 @@
   <xacro:macro name="dvl" params="parent_link dvl_name namespace">
     <!-- DVL Link -->
-    <link name="${namespace}_${dvl_name}_link">
+    <link name="${namespace}/${dvl_name}_link">
       <inertial>
         <mass value="0.105" />
@@ -112,7 +112,7 @@
     </link>
     <!-- Fixed joint to attach the DVL-->
-    <joint name="${namespace}_${dvl_name}_joint" type="fixed">
-      <parent link="${parent_link}" />
-      <child link="${namespace}_${dvl_name}_link" />
+    <joint name="${namespace}/${dvl_name}_joint" type="fixed">
+      <parent link="${parent_link}" />
+      <child link="${namespace}/${dvl_name}_link" />
       <origin xyz="0 0 -0.15" rpy="0 ${0.5*pi} 0" />
     </joint>
@@ -150,8 +150,8 @@
         <static_reference_frame>world</static_reference_frame>
         <!-- Declaring the links associated with individual sonar beams (see below)-->
-        <beam_link_name_0>${namespace}_${dvl_name}_sonar0_link</beam_link_name_0>
-        <beam_link_name_1>${namespace}_${dvl_name}_sonar1_link</beam_link_name_1>
-        <beam_link_name_2>${namespace}_${dvl_name}_sonar2_link</beam_link_name_2>
-        <beam_link_name_3>${namespace}_${dvl_name}_sonar3_link</beam_link_name_3>
+        <beam_link_name_0>${namespace}/${dvl_name}_sonar0_link</beam_link_name_0>
+        <beam_link_name_1>${namespace}/${dvl_name}_sonar1_link</beam_link_name_1>
+        <beam_link_name_2>${namespace}/${dvl_name}_sonar2_link</beam_link_name_2>
+        <beam_link_name_3>${namespace}/${dvl_name}_sonar3_link</beam_link_name_3>
         <!-- Declaring the individual sonar beam output ROS range topics -->
         <beam_topic_0>${dvl_name}_sonar0</beam_topic_0>
@@ -165,5 +165,5 @@
   <xacro:macro name="lidar" params="parent_link lidar_name namespace">
     <!-- Imaging Sonar Link -->
-    <link name="${namespace}_${lidar_name}_link">
+    <link name="${namespace}/${lidar_name}_link">
       <inertial>
         <origin xyz="0 0 0" rpy="0 0 0" />
@@ -173,11 +173,11 @@
     </link>
     <!-- Fixed Joint to Attach the Imaging Sonar -->
-    <joint name="${namespace}_${lidar_name}_joint" type="fixed">
-      <parent link="${parent_link}" />
-      <child link="${namespace}_${lidar_name}_link" />
+    <joint name="${namespace}/${lidar_name}_joint" type="fixed">
+      <parent link="${parent_link}" />
+      <child link="${namespace}/${lidar_name}_link" />
       <origin xyz="0 0 0.2" rpy="0 0 0" />
     </joint>
     <!-- Imaging Sonar Sensor -->
-    <gazebo reference="${namespace}_${lidar_name}_link">
+    <gazebo reference="${namespace}/${lidar_name}_link">
       <sensor type="ray" name="${lidar_name}_sensor">
         <pose> 0 0 0 0 0 0 </pose>
@@ -201,5 +201,5 @@
         <plugin filename="libgazebo_ros_laser.so" name="imaging_sonar">
           <topicName>${namespace}/scan</topicName>
-          <frameName>${namespace}_${lidar_name}_link</frameName>
+          <frameName>${namespace}/${lidar_name}_link</frameName>
         </plugin>
       </sensor>
@@ -209,5 +209,5 @@
   <xacro:macro name="altimeter" params="parent_link altimeter_name namespace">
     <!-- Altimeter Sonar Link -->
-    <link name="${namespace}_${altimeter_name}_link">
+    <link name="${namespace}/${altimeter_name}_link">
       <inertial>
         <origin xyz="0 0 0" rpy="0 0 0" />
@@ -217,11 +217,11 @@
     </link>
     <!-- Fixed Joint to Attach the Altimeter Sonar -->
-    <joint name="${namespace}_${altimeter_name}_joint" type="fixed">
-      <parent link="${parent_link}" />
-      <child link="${namespace}_${altimeter_name}_link" />
+    <joint name="${namespace}/${altimeter_name}_joint" type="fixed">
+      <parent link="${parent_link}" />
+      <child link="${namespace}/${altimeter_name}_link" />
       <origin xyz="0 0 0" rpy="0 ${0.5*pi} 0" />
     </joint>
     <!-- Altimaeter Sonar Sensor -->
-    <gazebo reference="${namespace}_${altimeter_name}_link">
+    <gazebo reference="${namespace}/${altimeter_name}_link">
       <sensor type="ray" name="${altimeter_name}_sensor">
         <pose> 0 0 0 0 0 0 </pose>
@@ -248,5 +248,5 @@
           <updateRate>10</updateRate>
           <topicName>${namespace}/depth</topicName>
-          <frameName>${namespace}_${altimeter_name}_link</frameName>
+          <frameName>${namespace}/${altimeter_name}_link</frameName>
           <fov>0.05</fov>
           <radiation>ultrasound</radiation>

File: urdf/thruster_snippets.xacro (robot description, xacro)
@@ -77,11 +77,11 @@
             *dynamics
             *conversion">
-    <joint name="${namespace}_thruster_${thruster_id}_joint" type="continuous">
+    <joint name="${namespace}/thruster_${thruster_id}_joint" type="continuous">
       <xacro:insert_block name="origin"/>
       <axis xyz="1 0 0"/>
       <parent link="${parent_link}"/>
-      <child link="${namespace}_thruster_${thruster_id}"/>
+      <child link="${namespace}/thruster_${thruster_id}"/>
     </joint>
-    <link name="${namespace}_thruster_${thruster_id}">
+    <link name="${namespace}/thruster_${thruster_id}">
       <xacro:box_inertial x="0" y="0" z="0" mass="0.001">
         <origin xyz="0 0 0" rpy="0 0 0"/>
@@ -104,6 +104,6 @@
     <gazebo>
       <plugin name="${namespace}_${thruster_id}_thruster_model" filename="libuuv_thruster_ros_plugin.so">
-        <linkName>${namespace}_thruster_${thruster_id}</linkName>
-        <jointName>${namespace}_thruster_${thruster_id}_joint</jointName>
+        <linkName>${namespace}/thruster_${thruster_id}</linkName>
+        <jointName>${namespace}/thruster_${thruster_id}_joint</jointName>
         <thrusterID>${thruster_id}</thrusterID>
         <xacro:insert_block name="dynamics"/>
@@ -111,5 +111,5 @@
       </plugin>
     </gazebo>
-    <gazebo reference="${namespace}_thruster_${thruster_id}">
+    <gazebo reference="${namespace}/thruster_${thruster_id}">
       <selfCollide>false</selfCollide>
     </gazebo>

Commit message: Update barracuda.xacro

File: urdf/barracuda.xacro (robot description, xacro)
@@ -42,4 +42,36 @@
     <xacro:include filename="$(find barracuda_description)/urdf/depth_camera.xacro"/>
     <xacro:depth_camera parent_link="$(arg namespace)/barracuda_link" namespace="$(arg namespace)"/>
+    <!--right top-->
+    <xacro:thruster_macro thruster_id="0">
+      <origin xyz="0.0 0.322 0.1535" rpy="${90*d2r} ${90*d2r} ${180*d2r}"/>
+    </xacro:thruster_macro>
+    <!--right mid-->
+    <xacro:thruster_macro thruster_id="1">
+      <origin xyz="-0.00525 0.43515 0.0" rpy="${90*d2r} 0 ${180*d2r}"/>
+    </xacro:thruster_macro>
+    <!--left top-->
+    <xacro:thruster_macro thruster_id="2">
+      <origin xyz="0.0 -0.322 0.1535" rpy="${-90*d2r} ${90*d2r} ${180*d2r}"/>
+    </xacro:thruster_macro>
+    <!--left mid-->
+    <xacro:thruster_macro thruster_id="3">
+      <origin xyz="-0.00525 -0.43515 0.0" rpy="${90*d2r} 0 ${180*d2r}"/>
+    </xacro:thruster_macro>
+    <!--front left-->
+    <xacro:thruster_macro thruster_id="4">
+      <origin xyz="-0.30916 -0.36341 0.0" rpy="${-90*d2r} ${135*d2r} ${131.51*d2r}"/>
+    </xacro:thruster_macro>
+    <!--back left-->
+    <xacro:thruster_macro thruster_id="5">
+      <origin xyz="0.30916 -0.36341 0.0" rpy="${-90*d2r} ${45*d2r} ${-131.51*d2r}"/>
+    </xacro:thruster_macro>
+    <!--front right-->
+    <xacro:thruster_macro thruster_id="6">
+      <origin xyz="-0.30916 0.36341 0.0" rpy="${90*d2r} ${135*d2r} ${-131.51*d2r}"/>
+    </xacro:thruster_macro>
+    <!--back right-->
+    <xacro:thruster_macro thruster_id="7">
+      <origin xyz="0.30916 0.36341 0.0" rpy="${-45*d2r} ${45*d2r} ${131.51*d2r}"/>
+    </xacro:thruster_macro>
     <gazebo>
         <plugin name="uuv_plugin" filename="libuuv_underwater_object_ros_plugin.so">
@@ -102,36 +134,4 @@
         </xacro:thruster_module_first_order_basic_fcn_macro>
     </xacro:macro>
-    <!--right top-->
-    <xacro:thruster_macro thruster_id="0">
-      <origin xyz="0.0 0.322 0.1535" rpy="${90*d2r} ${90*d2r} ${180*d2r}"/>
-    </xacro:thruster_macro>
-    <!--right mid-->
-    <xacro:thruster_macro thruster_id="1">
-      <origin xyz="-0.00525 0.43515 0.0" rpy="${90*d2r} 0 ${180*d2r}"/>
-    </xacro:thruster_macro>
-    <!--left top-->
-    <xacro:thruster_macro thruster_id="2">
-      <origin xyz="0.0 -0.322 0.1535" rpy="${-90*d2r} ${90*d2r} ${180*d2r}"/>
-    </xacro:thruster_macro>
-    <!--left mid-->
-    <xacro:thruster_macro thruster_id="3">
-      <origin xyz="-0.00525 -0.43515 0.0" rpy="${90*d2r} 0 ${180*d2r}"/>
-    </xacro:thruster_macro>
-    <!--front left-->
-    <xacro:thruster_macro thruster_id="4">
-      <origin xyz="-0.30916 -0.36341 0.0" rpy="${-90*d2r} ${135*d2r} ${131.51*d2r}"/>
-    </xacro:thruster_macro>
-    <!--back left-->
-    <xacro:thruster_macro thruster_id="5">
-      <origin xyz="0.30916 -0.36341 0.0" rpy="${-90*d2r} ${45*d2r} ${-131.51*d2r}"/>
-    </xacro:thruster_macro>
-    <!--front right-->
-    <xacro:thruster_macro thruster_id="6">
-      <origin xyz="-0.30916 0.36341 0.0" rpy="${90*d2r} ${135*d2r} ${-131.51*d2r}"/>
-    </xacro:thruster_macro>
-    <!--back right-->
-    <xacro:thruster_macro thruster_id="7">
-      <origin xyz="0.30916 0.36341 0.0" rpy="${-45*d2r} ${45*d2r} ${131.51*d2r}"/>
-    </xacro:thruster_macro>
     <!-- Default joint state publisher -->
     <gazebo>
