Commit message: fix bug

File: urdf/barracuda.xacro (robot description, xacro)
@@ -42,4 +42,15 @@
     <xacro:include filename="$(find barracuda_description)/urdf/depth_camera.xacro"/>
     <xacro:depth_camera parent_link="$(arg namespace)/barracuda_link" namespace="$(arg namespace)"/>
+    <xacro:macro name="thruster_macro" params="thruster_id *origin">
+        <xacro:thruster_module_first_order_basic_fcn_macro
+            namespace="$(arg namespace)"
+            thruster_id="${thruster_id}"
+            parent_link="$(arg namespace)/barracuda_link"
+            mesh_filename="${prop_mesh_file}"
+            dyn_time_constant="0.05"
+            rotor_constant="1">
+            <xacro:insert_block name="origin"/>
+        </xacro:thruster_module_first_order_basic_fcn_macro>
+    </xacro:macro>
     <!--right top-->
     <xacro:thruster_macro thruster_id="0">
@@ -123,15 +134,4 @@
     </gazebo>
     <!-- FROM MANTARAY NEED CHANGE -->
-    <xacro:macro name="thruster_macro" params="thruster_id *origin">
-        <xacro:thruster_module_first_order_basic_fcn_macro
-            namespace="$(arg namespace)"
-            thruster_id="${thruster_id}"
-            parent_link="$(arg namespace)/barracuda_link"
-            mesh_filename="${prop_mesh_file}"
-            dyn_time_constant="0.05"
-            rotor_constant="1">
-            <xacro:insert_block name="origin"/>
-        </xacro:thruster_module_first_order_basic_fcn_macro>
-    </xacro:macro>
     <!-- Default joint state publisher -->
     <gazebo>

Commit message: fix thruster order

File: urdf/barracuda.xacro (robot description, xacro)
@@ -42,47 +42,4 @@
     <xacro:include filename="$(find barracuda_description)/urdf/depth_camera.xacro"/>
     <xacro:depth_camera parent_link="$(arg namespace)/barracuda_link" namespace="$(arg namespace)"/>
-    <xacro:macro name="thruster_macro" params="thruster_id *origin">
-        <xacro:thruster_module_first_order_basic_fcn_macro
-            namespace="$(arg namespace)"
-            thruster_id="${thruster_id}"
-            parent_link="$(arg namespace)/barracuda_link"
-            mesh_filename="${prop_mesh_file}"
-            dyn_time_constant="0.05"
-            rotor_constant="1">
-            <xacro:insert_block name="origin"/>
-        </xacro:thruster_module_first_order_basic_fcn_macro>
-    </xacro:macro>
-    <!--right top-->
-    <xacro:thruster_macro thruster_id="0">
-      <origin xyz="0.0 0.322 0.1535" rpy="${90*d2r} ${90*d2r} ${180*d2r}"/>
-    </xacro:thruster_macro>
-    <!--right mid-->
-    <xacro:thruster_macro thruster_id="1">
-      <origin xyz="-0.00525 0.43515 0.0" rpy="${90*d2r} 0 ${180*d2r}"/>
-    </xacro:thruster_macro>
-    <!--left top-->
-    <xacro:thruster_macro thruster_id="2">
-      <origin xyz="0.0 -0.322 0.1535" rpy="${-90*d2r} ${90*d2r} ${180*d2r}"/>
-    </xacro:thruster_macro>
-    <!--left mid-->
-    <xacro:thruster_macro thruster_id="3">
-      <origin xyz="-0.00525 -0.43515 0.0" rpy="${90*d2r} 0 ${180*d2r}"/>
-    </xacro:thruster_macro>
-    <!--front left-->
-    <xacro:thruster_macro thruster_id="4">
-      <origin xyz="-0.30916 -0.36341 0.0" rpy="${-90*d2r} ${135*d2r} ${131.51*d2r}"/>
-    </xacro:thruster_macro>
-    <!--back left-->
-    <xacro:thruster_macro thruster_id="5">
-      <origin xyz="0.30916 -0.36341 0.0" rpy="${-90*d2r} ${45*d2r} ${-131.51*d2r}"/>
-    </xacro:thruster_macro>
-    <!--front right-->
-    <xacro:thruster_macro thruster_id="6">
-      <origin xyz="-0.30916 0.36341 0.0" rpy="${90*d2r} ${135*d2r} ${-131.51*d2r}"/>
-    </xacro:thruster_macro>
-    <!--back right-->
-    <xacro:thruster_macro thruster_id="7">
-      <origin xyz="0.30916 0.36341 0.0" rpy="${-45*d2r} ${45*d2r} ${131.51*d2r}"/>
-    </xacro:thruster_macro>
     <gazebo>
         <plugin name="uuv_plugin" filename="libuuv_underwater_object_ros_plugin.so">
@@ -133,5 +90,47 @@
         </plugin>
     </gazebo>
-    <!-- FROM MANTARAY NEED CHANGE -->
+    <xacro:macro name="thruster_macro" params="thruster_id *origin">
+        <xacro:thruster_module_first_order_basic_fcn_macro
+            namespace="$(arg namespace)"
+            thruster_id="${thruster_id}"
+            parent_link="$(arg namespace)/barracuda_link"
+            mesh_filename="${prop_mesh_file}"
+            dyn_time_constant="0.05"
+            rotor_constant="1">
+            <xacro:insert_block name="origin"/>
+        </xacro:thruster_module_first_order_basic_fcn_macro>
+    </xacro:macro>
+    <!--back left-->
+    <xacro:thruster_macro thruster_id="0">
+      <origin xyz="-0.30916 0.36341 0.0" rpy="${90*d2r} ${135*d2r} ${-131.51*d2r}"/>
+    </xacro:thruster_macro>
+    <!--left mid-->
+    <xacro:thruster_macro thruster_id="1">
+      <origin xyz="-0.00525 0.43515 0.0" rpy="${90*d2r} 0 ${180*d2r}"/>
+    </xacro:thruster_macro>
+    <!--left top-->
+    <xacro:thruster_macro thruster_id="2">
+      <origin xyz="0.0 0.322 0.1535" rpy="${90*d2r} ${90*d2r} ${180*d2r}"/>
+    </xacro:thruster_macro>
+    <!--front left-->
+    <xacro:thruster_macro thruster_id="3">
+      <origin xyz="0.30916 0.36341 0.0" rpy="${-45*d2r} ${45*d2r} ${131.51*d2r}"/>
+    </xacro:thruster_macro>
+    <!--front right-->
+    <xacro:thruster_macro thruster_id="4">
+      <origin xyz="0.30916 -0.36341 0.0" rpy="${-90*d2r} ${45*d2r} ${-131.51*d2r}"/>
+    </xacro:thruster_macro>
+    <!--right top-->
+    <xacro:thruster_macro thruster_id="5">
+      <origin xyz="0.0 -0.322 0.1535" rpy="${-90*d2r} ${90*d2r} ${180*d2r}"/>
+    </xacro:thruster_macro>
+    <!--right mid-->
+    <xacro:thruster_macro thruster_id="6">
+      <origin xyz="-0.00525 -0.43515 0.0" rpy="${90*d2r} 0 ${180*d2r}"/>
+    </xacro:thruster_macro>
+    <!--back right-->
+    <xacro:thruster_macro thruster_id="7">
+      <origin xyz="-0.30916 -0.36341 0.0" rpy="${-90*d2r} ${135*d2r} ${131.51*d2r}"/>
+    </xacro:thruster_macro>
     <!-- Default joint state publisher -->
     <gazebo>

Commit message: fix thruster order

File: urdf/barracuda.xacro (robot description, xacro)
@@ -101,11 +101,11 @@
         </xacro:thruster_module_first_order_basic_fcn_macro>
     </xacro:macro>
+    <!--left mid-->
+    <xacro:thruster_macro thruster_id="0">
+      <origin xyz="-0.00525 0.43515 0.0" rpy="${90*d2r} 0 ${180*d2r}"/>
+    </xacro:thruster_macro>
     <!--back left-->
-    <xacro:thruster_macro thruster_id="0">
+    <xacro:thruster_macro thruster_id="1">
       <origin xyz="-0.30916 0.36341 0.0" rpy="${90*d2r} ${135*d2r} ${-131.51*d2r}"/>
-    </xacro:thruster_macro>
-    <!--left mid-->
-    <xacro:thruster_macro thruster_id="1">
-      <origin xyz="-0.00525 0.43515 0.0" rpy="${90*d2r} 0 ${180*d2r}"/>
     </xacro:thruster_macro>
     <!--left top-->
@@ -117,11 +117,11 @@
       <origin xyz="0.30916 0.36341 0.0" rpy="${-45*d2r} ${45*d2r} ${131.51*d2r}"/>
     </xacro:thruster_macro>
+    <!--right top-->
+    <xacro:thruster_macro thruster_id="4">
+      <origin xyz="0.0 -0.322 0.1535" rpy="${-90*d2r} ${90*d2r} ${180*d2r}"/>
+    </xacro:thruster_macro>
     <!--front right-->
-    <xacro:thruster_macro thruster_id="4">
+    <xacro:thruster_macro thruster_id="5">
       <origin xyz="0.30916 -0.36341 0.0" rpy="${-90*d2r} ${45*d2r} ${-131.51*d2r}"/>
-    </xacro:thruster_macro>
-    <!--right top-->
-    <xacro:thruster_macro thruster_id="5">
-      <origin xyz="0.0 -0.322 0.1535" rpy="${-90*d2r} ${90*d2r} ${180*d2r}"/>
     </xacro:thruster_macro>
     <!--right mid-->

Commit message: Revert "fix thruster order"
This reverts commit a798f4fc1a595dad2468784d72b938c4d9f895be.

File: urdf/barracuda.xacro (robot description, xacro)
@@ -101,11 +101,11 @@
         </xacro:thruster_module_first_order_basic_fcn_macro>
     </xacro:macro>
+    <!--back left-->
+    <xacro:thruster_macro thruster_id="0">
+      <origin xyz="-0.30916 0.36341 0.0" rpy="${90*d2r} ${135*d2r} ${-131.51*d2r}"/>
+    </xacro:thruster_macro>
     <!--left mid-->
-    <xacro:thruster_macro thruster_id="0">
+    <xacro:thruster_macro thruster_id="1">
       <origin xyz="-0.00525 0.43515 0.0" rpy="${90*d2r} 0 ${180*d2r}"/>
-    </xacro:thruster_macro>
-    <!--back left-->
-    <xacro:thruster_macro thruster_id="1">
-      <origin xyz="-0.30916 0.36341 0.0" rpy="${90*d2r} ${135*d2r} ${-131.51*d2r}"/>
     </xacro:thruster_macro>
     <!--left top-->
@@ -117,11 +117,11 @@
       <origin xyz="0.30916 0.36341 0.0" rpy="${-45*d2r} ${45*d2r} ${131.51*d2r}"/>
     </xacro:thruster_macro>
+    <!--front right-->
+    <xacro:thruster_macro thruster_id="4">
+      <origin xyz="0.30916 -0.36341 0.0" rpy="${-90*d2r} ${45*d2r} ${-131.51*d2r}"/>
+    </xacro:thruster_macro>
     <!--right top-->
-    <xacro:thruster_macro thruster_id="4">
+    <xacro:thruster_macro thruster_id="5">
       <origin xyz="0.0 -0.322 0.1535" rpy="${-90*d2r} ${90*d2r} ${180*d2r}"/>
-    </xacro:thruster_macro>
-    <!--front right-->
-    <xacro:thruster_macro thruster_id="5">
-      <origin xyz="0.30916 -0.36341 0.0" rpy="${-90*d2r} ${45*d2r} ${-131.51*d2r}"/>
     </xacro:thruster_macro>
     <!--right mid-->

Commit message: update thruster

File: urdf/barracuda.xacro (robot description, xacro)
@@ -101,15 +101,15 @@
         </xacro:thruster_module_first_order_basic_fcn_macro>
     </xacro:macro>
+    <!--left top-->
+    <xacro:thruster_macro thruster_id="0">
+      <origin xyz="0.0 0.322 0.1535" rpy="${90*d2r} ${90*d2r} ${180*d2r}"/>
+    </xacro:thruster_macro>
     <!--back left-->
-    <xacro:thruster_macro thruster_id="0">
+    <xacro:thruster_macro thruster_id="1">
       <origin xyz="-0.30916 0.36341 0.0" rpy="${90*d2r} ${135*d2r} ${-131.51*d2r}"/>
     </xacro:thruster_macro>
     <!--left mid-->
-    <xacro:thruster_macro thruster_id="1">
+    <xacro:thruster_macro thruster_id="2">
       <origin xyz="-0.00525 0.43515 0.0" rpy="${90*d2r} 0 ${180*d2r}"/>
-    </xacro:thruster_macro>
-    <!--left top-->
-    <xacro:thruster_macro thruster_id="2">
-      <origin xyz="0.0 0.322 0.1535" rpy="${90*d2r} ${90*d2r} ${180*d2r}"/>
     </xacro:thruster_macro>
     <!--front left-->
@@ -117,15 +117,15 @@
       <origin xyz="0.30916 0.36341 0.0" rpy="${-45*d2r} ${45*d2r} ${131.51*d2r}"/>
     </xacro:thruster_macro>
+    <!--right mid-->
+    <xacro:thruster_macro thruster_id="4">
+      <origin xyz="-0.00525 -0.43515 0.0" rpy="${90*d2r} 0 ${180*d2r}"/>
+    </xacro:thruster_macro>
     <!--front right-->
-    <xacro:thruster_macro thruster_id="4">
+    <xacro:thruster_macro thruster_id="5">
       <origin xyz="0.30916 -0.36341 0.0" rpy="${-90*d2r} ${45*d2r} ${-131.51*d2r}"/>
     </xacro:thruster_macro>
     <!--right top-->
-    <xacro:thruster_macro thruster_id="5">
+    <xacro:thruster_macro thruster_id="6">
       <origin xyz="0.0 -0.322 0.1535" rpy="${-90*d2r} ${90*d2r} ${180*d2r}"/>
-    </xacro:thruster_macro>
-    <!--right mid-->
-    <xacro:thruster_macro thruster_id="6">
-      <origin xyz="-0.00525 -0.43515 0.0" rpy="${90*d2r} 0 ${180*d2r}"/>
     </xacro:thruster_macro>
     <!--back right-->

Commit message: test

File: urdf/barracuda.xacro (robot description, xacro)
@@ -74,7 +74,7 @@
     </xacro:thruster_macro>
     <!--back left-->
-    <xacro:thruster_macro thruster_id="5">
-      <origin xyz="0.30916 -0.36341 0.0" rpy="${-90*d2r} ${45*d2r} ${-131.51*d2r}"/>
-    </xacro:thruster_macro>
+    <!-- <xacro:thruster_macro thruster_id="5"> -->
+    <!--   <origin xyz="0.30916 -0.36341 0.0" rpy="${-90*d2r} ${45*d2r} ${-131.51*d2r}"/> -->
+    <!-- </xacro:thruster_macro> -->
     <!--front right-->
     <xacro:thruster_macro thruster_id="6">

Commit message: update

File: urdf/barracuda.xacro (robot description, xacro)
@@ -106,7 +106,7 @@
     </xacro:thruster_macro>
     <!--back left-->
-    <xacro:thruster_macro thruster_id="1">
-      <origin xyz="-0.30916 0.36341 0.0" rpy="${90*d2r} ${135*d2r} ${-131.51*d2r}"/>
-    </xacro:thruster_macro>
+    <!-- <xacro:thruster_macro thruster_id="1"> -->
+    <!--   <origin xyz="-0.30916 0.36341 0.0" rpy="${90*d2r} ${135*d2r} ${-131.51*d2r}"/> -->
+    <!-- </xacro:thruster_macro> -->
     <!--left mid-->
     <xacro:thruster_macro thruster_id="2">

Commit message: fixed thruster 3

File: urdf/barracuda.xacro (robot description, xacro)
@@ -67,5 +67,5 @@
     <!--left mid-->
     <xacro:thruster_macro thruster_id="3">
-      <origin xyz="-0.00525 -0.43515 0.0" rpy="${90*d2r} 0 ${180*d2r}"/>
+      <origin xyz="-0.00525 -0.43515 0.0" rpy="${-90*d2r} 0 ${180*d2r}"/>
     </xacro:thruster_macro>
     <!--front left-->

Commit message: Flip thruster orientations and add joint state publisher with GUI dependencies

File: urdf/barracuda.xacro (robot description, xacro)
@@ -103,33 +103,33 @@
     <!--left top-->
     <xacro:thruster_macro thruster_id="3">
-      <origin xyz="0.0 0.322 0.1535" rpy="${90*d2r} ${90*d2r} ${180*d2r}"/>
+      <origin xyz="0.0 0.322 0.1535" rpy="${90*d2r} ${-90*d2r} ${180*d2r}"/>
     </xacro:thruster_macro>
     <!--back left-->
     <xacro:thruster_macro thruster_id="2">
-      <origin xyz="-0.30916 0.36341 0.0" rpy="${90*d2r} ${135*d2r} ${-131.51*d2r}"/>
+      <origin xyz="-0.30916 0.36341 0.0" rpy="${90*d2r} ${-45*d2r} ${-131.51*d2r}"/>
     </xacro:thruster_macro>
     <!--left mid-->
     <xacro:thruster_macro thruster_id="1">
-      <origin xyz="-0.00525 0.43515 0.0" rpy="${90*d2r} 0 ${180*d2r}"/>
+      <origin xyz="-0.00525 0.43515 0.0" rpy="${90*d2r} ${180*d2r} ${180*d2r}"/>
     </xacro:thruster_macro>
     <!--front left-->
     <xacro:thruster_macro thruster_id="0">
-      <origin xyz="0.30916 0.36341 0.0" rpy="${-45*d2r} ${45*d2r} ${131.51*d2r}"/>
+      <origin xyz="0.30916 0.36341 0.0" rpy="${-45*d2r} ${-135*d2r} ${131.51*d2r}"/>
     </xacro:thruster_macro>
     <!--right mid-->
     <xacro:thruster_macro thruster_id="6">
-      <origin xyz="-0.00525 -0.43515 0.0" rpy="${90*d2r} 0 ${180*d2r}"/>
+      <origin xyz="-0.00525 -0.43515 0.0" rpy="${90*d2r} ${180*d2r} ${180*d2r}"/>
     </xacro:thruster_macro>
     <!--front right-->
     <xacro:thruster_macro thruster_id="7">
-      <origin xyz="0.30916 -0.36341 0.0" rpy="${-90*d2r} ${45*d2r} ${-131.51*d2r}"/>
+      <origin xyz="0.30916 -0.36341 0.0" rpy="${-90*d2r} ${-135*d2r} ${-131.51*d2r}"/>
     </xacro:thruster_macro>
     <!--right top-->
     <xacro:thruster_macro thruster_id="4">
-      <origin xyz="0.0 -0.322 0.1535" rpy="${-90*d2r} ${90*d2r} ${180*d2r}"/>
+      <origin xyz="0.0 -0.322 0.1535" rpy="${-90*d2r} ${-90*d2r} ${180*d2r}"/>
     </xacro:thruster_macro>
     <!--back right-->
     <xacro:thruster_macro thruster_id="5">
-      <origin xyz="-0.30916 -0.36341 0.0" rpy="${-90*d2r} ${135*d2r} ${131.51*d2r}"/>
+      <origin xyz="-0.30916 -0.36341 0.0" rpy="${-90*d2r} ${-45*d2r} ${131.51*d2r}"/>
     </xacro:thruster_macro>
     <!-- Default joint state publisher -->
